File: Hardware/Front.brd (EAGLE design)
At the start: 100 x 17 mm, 60 parts, among them IC3 MAX6951

Commit message: Add various parts
Parts:
- removed C14, C15, C16, C17, C18, C19: (no value), rcl:C0805
- removed U1: (no value), MyLib:EFM8BB10F(2/4/8)G-A-QFN20
- added Q1, Q2, Q3, Q4, Q5, Q6, Q9: BC847BS, transistor-small-signal:SOT363_PHILIPS
- added Q7: (no value), crystal-geyer_V1_0:2.0X1.6_KX-5
- added R17, R18, R19, R20, R21, R22, R23, R24, R25, R26, R27: (no value), rcl:R0402
- added TP1, TP2, TP3, TP4: TPB1,27, testpad:B1,27
- C1: value (none) -> 100n; device rcl:C0603 -> rcl:C0402
- C10, C4, C5, C6, C8, C9: device rcl:C0603 -> rcl:C0402
- C2: value (none) -> 22p; device rcl:C0603 -> rcl:C0402
- C3: value 100n -> 22p; device rcl:C0603 -> rcl:C0402
- IC3: value MAX6951 -> MEGA8-MI; device MyLib:QSOP16 -> atmel:MLF32-TH
- R1, R10, R11, R12, R13, R14, R15, R16, R2, R3, R4, R5, R6, R7, R8, R9: value 10k -> (none); device rcl:R0603 -> rcl:R0402
- moved R8 62.6 mm to (72.2, 4.80), turned to 0 degrees
- moved R9 60.2 mm to (72.2, 3.60), turned to 0 degrees
- moved R14 56.0 mm to (89.6, 10.4), turned to 270 degrees
- moved C1 29.6 mm to (9.40, -9.80), flipped to the top, turned to 0 degrees
- moved R15 25.5 mm to (31.6, -4.00), turned to 90 degrees
- moved R1 23.5 mm to (32.8, -4.00)
- moved R2 20.4 mm to (72.2, 12.0), turned to 0 degrees
- moved R16 20.1 mm to (-4.80, -2.60), flipped to the top, turned to 0 degrees
- moved R6 20.0 mm to (72.2, 7.20), turned to 0 degrees
- moved R4 19.6 mm to (72.2, 9.60), turned to 0 degrees
- moved IC3 18.4 mm to (11.6, 8.30), turned to 225 degrees
- moved C2 17.9 mm to (7.60, 12.8), turned to 270 degrees
- moved C8 17.5 mm to (-0.60, -5.60), turned to 90 degrees
- moved R7 17.1 mm to (72.2, 6.00)
- moved R3 17.0 mm to (72.2, 10.8)
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Connections:
- removed net C2CK: R1.1, U$2.P$4, U1.P$5
- removed net FRONT_INT/C2D: U$2.P$3, U1.P$6
- removed net N$37: LED_PWR.C, U1.P$16
- removed net N$6: LED_CHG.A, R15.1
- removed net SPI_!CS: IC3.15, U1.P$19
- removed net SPI_CLK: IC3.2, U1.P$2
- removed net SPI_MOSI: IC3.1, U1.P$20
- removed net UART_RX: U$2.P$5, U1.P$17
- removed net UART_TX: U$2.P$6, U1.P$18
- new net ISP_RESET: C1.1, IC3.29, R24.2, TP4.TP
- new net N$10: IC3.26, Q2.5
- new net N$11: IC3.27, Q3.2
- new net N$12: IC3.28, Q3.5
- new net N$13: IC3.19, Q4.2
- new net N$16: IC3.22, Q4.5
- new net N$17: C2.2, IC3.7, Q7.3
- new net N$18: IC3.14, Q9.5
- new net N$19: IC3.13, Q9.2
- new net N$20: IC3.12, Q6.5
- new net N$21: IC3.11, Q6.2
- new net N$22: IC3.10, Q5.5
- new net N$23: IC3.9, Q5.2
- new net N$24: IC3.2, R16.1
- new net N$25: IC3.1, R25.1
- new net N$26: IC3.23, Q1.2
- new net N$27: C3.2, IC3.8, Q7.1
- new net N$28: IC3.32, R26.1
- new net N$29: IC3.16, R27.1, TP2.TP
- new net UART_IN: IC3.30, U$2.P$6
- new net UART_OUT: IC3.31, U$2.P$5
- net +3V3: now also IC3.18, IC3.20, IC3.4, IC3.6, Q5.1, Q5.4, Q6.1, Q6.4, Q9.1, Q9.4, R10.1, R12.1, R14.1, R18.1, R20.1, R22.1, R24.1; no longer C14.1, C15.1, C16.1, C17.1, C18.1, C19.1, C2.1, C3.1, IC3.16, R1.2, R10.2, R12.2, R15.2, R16.2, R2.2, R4.2, R6.2, R8.2, U1.P$4
- net BTN_DWN: now also R21.2, R26.2; no longer R13.2, U1.P$11
- net BTN_PWR: now also R16.2, R23.2; no longer R9.2, U1.P$13
- net BTN_RAW_DWN: now also R22.2, R23.1, S_PWR.1, S_PWR.2; no longer R12.1, R13.1, S_DOWN.1, S_DOWN.2
- net BTN_RAW_PWR: now also R20.2, R21.1, S_DOWN.1, S_DOWN.2; no longer R8.1, R9.1, S_PWR.1, S_PWR.2
- net BTN_RAW_UP: now also R18.2, R19.1; no longer R10.1, R11.1
- net BTN_UP: now also R19.2, R25.2; no longer R11.2, U1.P$7
- net ENC_A: now also R1.2, R11.2; no longer R3.2, U1.P$10
- net ENC_B: now also R13.2, R27.2; no longer R5.2, U1.P$9
- net ENC_C: now also R15.2, R17.2; no longer R7.2, U1.P$8
- net ENC_RAW_A: now also R10.2, R11.1; no longer R2.1, R3.1
- net ENC_RAW_B: now also R12.2, R13.1; no longer R4.1, R5.1
- net ENC_RAW_C: now also R14.2, R17.1; no longer R6.1, R7.1
- net GND: now also C2.1, C3.1, IC3.21, IC3.3, IC3.5, IC3.TH, Q1.1, Q1.4, Q2.1, Q2.4, Q3.1, Q3.4, Q4.1, Q4.4; no longer C14.2, C15.2, C16.2, C17.2, C18.2, C19.2, C2.2, C3.2, IC3.8, R14.1, U1.P$12, U1.P$3, U1.PAD
- net N$1: no longer IC3.6
- net N$14: no longer IC3.4
- net N$15: now also IC3.15, R15.1, TP1.TP; no longer LED_PWR.A, R16.1
- net N$2: no longer IC3.12
- net N$3: no longer IC3.11
- net N$36: no longer IC3.3
- net N$4: no longer IC3.10
- net N$5: now also IC3.24, Q1.5; no longer IC3.7, R14.2
- net N$51: no longer IC3.14
- net N$53: no longer IC3.13
- net N$7: now also IC3.17, R1.1, TP3.TP; no longer LED_CHG.C, U1.P$15
- net N$8: now also IC3.25, Q2.2; no longer C1.1, IC3.9
- net N$9: no longer IC3.5
Routing:
- net BTN_UP: track 90.6 -> 0.00 mm, vias 2 -> 0
- net ENC_C: track 86.0 -> 0.00 mm, vias 2 -> 0
- net BTN_DWN: track 85.2 -> 0.00 mm, vias 2 -> 0
- net ENC_B: track 84.7 -> 0.00 mm, vias 2 -> 0
- net ENC_A: track 83.3 -> 0.00 mm, vias 2 -> 0
- net N$51: track 79.9 -> 0.00 mm, vias 6 -> 0
- net N$1: track 78.6 -> 0.00 mm, vias 6 -> 0
- net N$36: track 77.9 -> 0.00 mm, vias 6 -> 0
- net N$2: track 71.8 -> 0.00 mm, vias 7 -> 0
- net N$9: track 71.7 -> 0.00 mm, vias 6 -> 0
- net N$53: track 71.6 -> 0.00 mm, vias 6 -> 0
- net N$3: track 70.7 -> 0.00 mm, vias 5 -> 0
- net N$4: track 70.1 -> 0.00 mm, vias 6 -> 0
- net N$14: track 70.0 -> 0.00 mm, vias 6 -> 0
- net +3V3: track 31.6 -> 0.00 mm, vias 20 -> 0
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
Commit message: Add various parts
Parts:
- removed C1, C4, C5, C6: 100n, rcl:C0402
- removed C2, C3: 22p, rcl:C0402
- removed IC3: MEGA8-MI, atmel:MLF32-TH
- removed LED_S1: (no value), led:CHIPLED_0603
- removed Q1, Q2, Q3, Q4, Q5, Q6, Q9: BC847BS, transistor-small-signal:SOT363_PHILIPS
- removed Q7: (no value), crystal-geyer_V1_0:2.0X1.6_KX-5
- removed R10, R11, R12, R13, R14, R15, R16, R17, R24, R25, R26, R27, R9: (no value), rcl:R0402
- removed TP1, TP2, TP3, TP4: TPB1,27, testpad:B1,27
- removed U$2: JST-SH-8-SMT, MyLib:JST-SH-8-SMT
- removed U$3: JST-SH-4-SMT, MyLib:JST-SH-4-SMT
- removed U$4, U$5, U$6, U$7: ACSC02-41SURKWA-F01, MyLib:ACSC02
- added D3, U$10, U$11, U$9: HDSP-C3E1, MyLib:7SEG_THT
- added X2: PHB_1MM27_2X10_SNS, _hhn_con_pinhead_box_1mm27:PHB_1MM27_2X10_SNS
- moved R20 60.5 mm to (32.2, -6.20), turned to 180 degrees
- moved R18 59.9 mm to (32.4, 6.20), turned to 180 degrees
- moved R19 56.6 mm to (34.6, 6.20), turned to 180 degrees
- moved R21 56.0 mm to (34.6, -6.20), turned to 180 degrees
- moved C9 52.6 mm to (37.4, 6.20), turned to 180 degrees
- moved LED_S2 51.0 mm to (16.0, -6.00), turned to 90 degrees
- moved LED_S3 50.9 mm to (16.0, -4.29)
- moved C10 50.9 mm to (37.4, -6.20), turned to 180 degrees
- moved LED_S4 50.9 mm to (16.0, -2.57)
- moved LED_S5 50.9 mm to (16.0, -0.86)
- moved LED_S6 50.8 mm to (16.0, 0.86)
- moved LED_S7 50.8 mm to (16.0, 2.57)
- moved LED_S8 50.8 mm to (16.0, 4.29)
- moved LED_AM 50.7 mm to (-24.0, -2.00)
- moved LED_CHG 50.7 mm to (-44.0, -4.00)
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Connections:
- removed net BTN_DWN: C10.1, R21.2, R26.2
- removed net BTN_RAW_DWN: R22.2, R23.1, S_PWR.1, S_PWR.2
- removed net ENC_A: C4.1, R1.2, R11.2
- removed net ENC_B: C5.1, R13.2, R27.2
- removed net ENC_C: C6.1, R15.2, R17.2
- removed net ENC_RAW_A: R10.2, R11.1, U$3.P$1
- removed net ENC_RAW_B: R12.2, R13.1, U$3.P$2
- removed net ENC_RAW_C: R14.2, R17.1, U$3.P$3
- removed net ISP_RESET: C1.1, IC3.29, R24.2, TP4.TP
- removed net N$10: IC3.26, Q2.5
- removed net N$11: IC3.27, Q3.2
- removed net N$12: IC3.28, Q3.5
- removed net N$13: IC3.19, Q4.2
- removed net N$14: LED_LSB.A, LED_S6.A, U$4.G, U$5.G, U$6.CC@1, U$6.CC@2, U$7.F
- removed net N$15: IC3.15, R15.1, TP1.TP
- removed net N$16: IC3.22, Q4.5
- removed net N$17: C2.2, IC3.7, Q7.3
- removed net N$18: IC3.14, Q9.5
- removed net N$19: IC3.13, Q9.2
- removed net N$20: IC3.12, Q6.5
- removed net N$21: IC3.11, Q6.2
- removed net N$22: IC3.10, Q5.5
- removed net N$23: IC3.9, Q5.2
- removed net N$24: IC3.2, R16.1
- removed net N$25: IC3.1, R25.1
- removed net N$26: IC3.23, Q1.2
- removed net N$27: C3.2, IC3.8, Q7.1
- removed net N$28: IC3.32, R26.1
- removed net N$29: IC3.16, R27.1, TP2.TP
- removed net N$36: LED_AM.A, LED_S5.A, U$4.F, U$5.F, U$6.F, U$7.CC@1, U$7.CC@2
- removed net N$51: LED_AM.C, LED_CW.C, LED_DBG.C, LED_LSB.C, LED_PC.C, LED_S4.A, LED_USB.C, U$4.E, U$5.E, U$6.E, U$7.E
- removed net N$53: LED_DBG.A, LED_S1.C, LED_S2.C, LED_S3.C, LED_S4.C, LED_S5.C, LED_S6.C, LED_S7.C, LED_S8.C, U$4.D, U$5.D, U$6.D, U$7.D
- removed net N$9: LED_S7.A, LED_USB.A, U$4.DP, U$5.CC@1, U$5.CC@2, U$6.G, U$7.G
- removed net UART_IN: IC3.30, U$2.P$6
- removed net UART_OUT: IC3.31, U$2.P$5
- new net BTN_DN: C10.1, R21.2
- new net BTN_RAW_DN: R20.2, R21.1, S_DOWN.1, S_DOWN.2
- new net N$6: D3.P$8, R6.2, U$10.P$8, U$11.P$8, U$9.P$8
- new net N$77: LED_AM.A, LED_CHG.A, LED_CW.A, LED_DBG.A, LED_LSB.A, LED_PC.A, LED_PWR.A, LED_USB.A
- new net N$82: LED_S2.A, LED_S3.A, LED_S4.A, LED_S5.A, LED_S6.A, LED_S7.A, LED_S8.A, LED_S9.A
- net +3V3: no longer IC3.18, IC3.20, IC3.4, IC3.6, Q5.1, Q5.4, Q6.1, Q6.4, Q9.1, Q9.4, R10.1, R12.1, R14.1, R24.1, U$2.P$1, U$2.P$2
- net BTN_PWR: no longer R16.2
- net BTN_RAW_PWR: now also R22.2, R23.1, S_PWR.1, S_PWR.2; no longer R20.2, R21.1, S_DOWN.1, S_DOWN.2
- net BTN_UP: no longer R25.2
- net GND: no longer C1.2, C2.1, C3.1, C4.2, C5.2, C6.2, IC3.21, IC3.3, IC3.5, IC3.TH, Q1.1, Q1.4, Q2.1, Q2.4, Q3.1, Q3.4, Q4.1, Q4.4, U$2.P$7, U$2.P$8, U$3.P$4
- net N$1: now also D3.P$7, R1.2, U$10.P$7, U$11.P$7, U$9.P$7; no longer LED_CW.A, LED_S8.A, U$4.CC@1, U$4.CC@2, U$5.DP, U$6.DP, U$7.DP
- net N$2: now also D3.P$3, R2.2, U$10.P$3, U$11.P$3, U$9.P$3; no longer LED_PC.A, LED_S3.A, LED_S9.C, U$4.C, U$5.C, U$6.C, U$7.C
- net N$3: now also D3.P$2, R3.2, U$10.P$2, U$11.P$2, U$9.P$2; no longer LED_S2.A, LED_S9.A, U$4.B, U$5.B, U$6.B, U$7.B
- net N$4: now also D3.P$4, R4.2, U$10.P$4, U$11.P$4, U$9.P$4; no longer LED_S1.A, U$4.A, U$5.A, U$6.A, U$7.A
- net N$5: now also D3.P$5, R5.2, U$10.P$5, U$11.P$5, U$9.P$5; no longer IC3.24, Q1.5
- net N$7: now also D3.P$9, R7.2, U$10.P$9, U$11.P$9, U$9.P$9; no longer IC3.17, R1.1, TP3.TP
- net N$8: now also D3.P$10, R8.2, U$10.P$10, U$11.P$10, U$9.P$10; no longer IC3.25, Q2.2
Routing:
- net N$12: track 23.3 -> 182.4 mm
- net N$14: track 0.00 -> 32.8 mm
- net N$9: track 0.00 -> 30.6 mm
- net N$13: track 14.0 -> 33.0 mm
- net N$16: track 16.0 -> 0.00 mm
- net N$26: track 13.7 -> 0.00 mm
- net N$10: track 18.4 -> 30.6 mm
- net N$11: track 18.2 -> 30.4 mm
- net N$23: track 10.9 -> 0.00 mm
- net N$22: track 10.5 -> 0.00 mm
- net N$21: track 10.2 -> 0.00 mm
- net N$20: track 9.78 -> 0.00 mm
- net N$8: track 16.5 -> 6.94 mm, vias 0 -> 4
- net N$19: track 9.41 -> 0.00 mm
- net N$18: track 9.04 -> 0.00 mm
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Other:
- board text added: "S2"
- board text removed: "S1"

Commit message: Advance layout bottom
Changed lines of the file:
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@@
 </signal>
 <signal name="N$14">
-<wire x1="13.2" y1="6.8" x2="-19.6" y2="6.8" width="0.4" layer="16"/>
+<wire x1="13.4" y1="6.8" x2="-19.4" y2="6.8" width="0.4" layer="16"/>
 </signal>
 </signals>
