File: Hardware/Front.sch (EAGLE design)
At the start: 60 parts, among them IC3 MAX6951

Commit message: Finish version 0.1 of front
Other:
- moved on the sheet: U$1

Commit message: Add various parts
Parts:
- removed C14, C15, C16, C17, C18, C19: (no value), rcl:C-EUC0805
- removed U1: (no value), MyLib:EFM8BB10F(2/4/8)G-A-QFN20
- added Q1, Q2, Q3, Q4, Q5, Q6, Q9: BC847BS, transistor-small-signal:BC847BS
- added Q7: (no value), crystal-geyer_V1_0:KX-5
- added R17, R18, R19, R20, R21, R22, R23, R24, R25, R26, R27: (no value), rcl:R-EU_R0402
- added TP1, TP2, TP3, TP4: TPB1,27, testpad:TPB1,27
- C1: value (none) -> 100n; device rcl:C-EUC0603 -> rcl:C-EUC0402; OC_FARNELL (none) -> unknown
- C10, C4, C5, C6, C8, C9: device rcl:C-EUC0603 -> rcl:C-EUC0402; OC_FARNELL (none) -> unknown
- C2: value (none) -> 22p; device rcl:C-EUC0603 -> rcl:C-EUC0402; OC_FARNELL (none) -> unknown
- C3: value 100n -> 22p; device rcl:C-EUC0603 -> rcl:C-EUC0402; OC_FARNELL (none) -> unknown
- IC3: value MAX6951 -> MEGA8-MI; device MyLib:MAX6951 -> atmel:MEGA8-MI
- LED_AM, LED_CHG, LED_CW, LED_DBG, LED_LSB, LED_PC, LED_PWR, LED_S1, LED_S2, LED_S3, LED_S4, LED_S5, LED_S6, LED_S7, LED_S8, LED_S9, LED_USB: MF (none) -> ROHM; MPN (none) -> SML-E12UWT86; OC_FARNELL (none) -> 2762561
- R1, R10, R11, R12, R13, R14, R15, R16, R2, R3, R4, R5, R6, R7, R8, R9: value 10k -> (none); device rcl:R-EU_R0603 -> rcl:R-EU_R0402
- S_DOWN, S_PWR, S_UP, U$1, U$2, U$3, U$4, U$5, U$6, U$7: OC_FARNELL (none) -> unknown
Connections:
- removed net C2CK: R1.1, U$2G$4.S, U1.!RST!/C2CK
- removed net FRONT_INT/C2D: U$2G$3.S, U1.C2D/P2.7
- removed net N$37: LED_PWR.C, U1.P0.6
- removed net N$6: LED_CHG.A, R15.1
- removed net SPI_!CS: IC3.!CS, U1.P0.3
- removed net SPI_CLK: IC3.CLK, U1.P0.0
- removed net SPI_MOSI: IC3.DIN, U1.P0.2
- removed net UART_RX: U$2G$5.S, U1.P0.5
- removed net UART_TX: U$2G$6.S, U1.P0.4
- new net ISP_RESET: C1.1, IC3.PC6(/RESET), R24.2, TP4.TP
- new net N$10: IC3.PC3(ADC3), Q2B.B
- new net N$11: IC3.PC4(ADC4/SDA), Q3A.B
- new net N$12: IC3.PC5(ADC5/SCL), Q3B.B
- new net N$13: IC3.ADC6, Q4A.B
- new net N$16: IC3.ADC7, Q4B.B
- new net N$17: C2.2, IC3.PB6(XTAL1/TOSC1), Q7.2
- new net N$18: IC3.PB2(SS/OC1B), Q9B.B
- new net N$19: IC3.PB1(OC1A), Q9A.B
- new net N$20: IC3.PB0(ICP), Q6B.B
- new net N$21: IC3.PD7(AIN1), Q6A.B
- new net N$22: IC3.PD6(AIN0), Q5B.B
- new net N$23: IC3.PD5(T1), Q5A.B
- new net N$24: IC3.PD4(XCK/T0), R16.1
- new net N$25: IC3.PD3(INT1), R25.1
- new net N$26: IC3.PC0(ADC0), Q1A.B
- new net N$27: C3.2, IC3.PB7(XTAL2/TOSC2), Q7.1
- new net N$28: IC3.PD2(INT0), R26.1
- new net N$29: IC3.PB4(MISO), R27.1, TP2.TP
- new net UART_IN: IC3.PD0(RXD), U$2G$6.S
- new net UART_OUT: IC3.PD1(TXD), U$2G$5.S
- net +3V3: now also IC3.AREF, IC3.AVCC, IC3.VCC@1, IC3.VCC@2, Q5A.E, Q5B.E, Q6A.E, Q6B.E, Q9A.E, Q9B.E, R10.1, R12.1, R14.1, R18.1, R20.1, R22.1, R24.1; no longer C14.1, C15.1, C16.1, C17.1, C18.1, C19.1, C2.1, C3.1, IC3.VCC, R1.2, R10.2, R12.2, R15.2, R16.2, R2.2, R4.2, R6.2, R8.2, U1.VDD
- net BTN_DWN: now also R21.2, R26.2; no longer R13.2, U1.P1.2
- net BTN_PWR: now also R16.2, R23.2; no longer R9.2, U1.P1.1
- net BTN_RAW_DWN: now also R22.2, R23.1, S_PWR.1, S_PWR.2; no longer R12.1, R13.1, S_DOWN.1, S_DOWN.2
- net BTN_RAW_PWR: now also R20.2, R21.1, S_DOWN.1, S_DOWN.2; no longer R8.1, R9.1, S_PWR.1, S_PWR.2
- net BTN_RAW_UP: now also R18.2, R19.1; no longer R10.1, R11.1
- net BTN_UP: now also R19.2, R25.2; no longer R11.2, U1.P1.6
- net ENC_A: now also R1.2, R11.2; no longer R3.2, U1.P1.3
- net ENC_B: now also R13.2, R27.2; no longer R5.2, U1.P1.4
- net ENC_C: now also R15.2, R17.2; no longer R7.2, U1.P1.5
- net ENC_RAW_A: now also R10.2, R11.1; no longer R2.1, R3.1
- net ENC_RAW_B: now also R12.2, R13.1; no longer R4.1, R5.1
- net ENC_RAW_C: now also R14.2, R17.1; no longer R6.1, R7.1
- net GND: now also C2.1, C3.1, IC3.GND@1, IC3.GND@2, IC3.THERMAL, Q1A.E, Q1B.E, Q2A.E, Q2B.E, Q3A.E, Q3B.E, Q4A.E, Q4B.E; no longer C14.2, C15.2, C16.2, C17.2, C18.2, C19.2, C2.2, C3.2, R14.1, U1.GND
- net N$1: no longer IC3.DIG0/SEG0
- net N$14: no longer IC3.DIG2/SEG2
- net N$15: now also IC3.PB3(MOSI/OC2), R15.1, TP1.TP; no longer LED_PWR.A, R16.1
- net N$2: no longer IC3.DIG6/SEG6
- net N$3: no longer IC3.DIG7/SEG7
- net N$36: no longer IC3.DIG3/SEG3
- net N$4: no longer IC3.DIG8
- net N$5: now also IC3.PC1(ADC1), Q1B.B; no longer IC3.ISET, R14.2
- net N$51: no longer IC3.DIG4/SEG4
- net N$53: no longer IC3.DIG5/SEG5
- net N$7: now also IC3.PB5(SCK), R1.1, TP3.TP; no longer LED_CHG.C, U1.P0.7
- net N$8: now also IC3.PC2(ADC2), Q2A.B; no longer C1.1, IC3.OSC
- net N$9: no longer IC3.DIG1/SEG1
Other:
- moved on the sheet: C1, C10, C2, C3, C4, C5, C6, C8, C9, LED_AM, LED_CHG, LED_CW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

Commit message: Add various parts
Parts:
- removed C1, C4, C5, C6: 100n, rcl:C-EUC0402
- removed C2, C3: 22p, rcl:C-EUC0402
- removed IC3: MEGA8-MI, atmel:MEGA8-MI
- removed LED_S1: (no value), led:LEDCHIPLED_0603
- removed Q1, Q2, Q3, Q4, Q5, Q6, Q9: BC847BS, transistor-small-signal:BC847BS
- removed Q7: (no value), crystal-geyer_V1_0:KX-5
- removed R10, R11, R12, R13, R14, R15, R16, R17, R24, R25, R26, R27, R9: (no value), rcl:R-EU_R0402
- removed TP1, TP2, TP3, TP4: TPB1,27, testpad:TPB1,27
- removed U$2: JST-SH-8-SMT, MyLib:JST-SH-8-SMT
- removed U$3: JST-SH-4-SMT, MyLib:JST-SH-4-SMT
- removed U$4, U$5, U$6, U$7: ACSC02-41SURKWA-F01, MyLib:ACSC02-41SURKWA-F01
- added D3, U$10, U$11, U$9: HDSP-C3E1, MyLib:HDSP-C3E1
- added X2: PHB_1MM27_2X10_SNS, _hhn_con_pinhead_box_1mm27:PHB_1MM27_2X10_SNS
Connections:
- removed net BTN_DWN: C10.1, R21.2, R26.2
- removed net BTN_RAW_DWN: R22.2, R23.1, S_PWR.1, S_PWR.2
- removed net ENC_A: C4.1, R1.2, R11.2
- removed net ENC_B: C5.1, R13.2, R27.2
- removed net ENC_C: C6.1, R15.2, R17.2
- removed net ENC_RAW_A: R10.2, R11.1, U$3G$1.S
- removed net ENC_RAW_B: R12.2, R13.1, U$3G$2.S
- removed net ENC_RAW_C: R14.2, R17.1, U$3G$3.S
- removed net ISP_RESET: C1.1, IC3.PC6(/RESET), R24.2, TP4.TP
- removed net N$10: IC3.PC3(ADC3), Q2B.B
- removed net N$11: IC3.PC4(ADC4/SDA), Q3A.B
- removed net N$12: IC3.PC5(ADC5/SCL), Q3B.B
- removed net N$13: IC3.ADC6, Q4A.B
- removed net N$14: LED_LSB.A, LED_S6.A, U$4.G, U$5.G, U$6.CC, U$7.F
- removed net N$15: IC3.PB3(MOSI/OC2), R15.1, TP1.TP
- removed net N$16: IC3.ADC7, Q4B.B
- removed net N$17: C2.2, IC3.PB6(XTAL1/TOSC1), Q7.2
- removed net N$18: IC3.PB2(SS/OC1B), Q9B.B
- removed net N$19: IC3.PB1(OC1A), Q9A.B
- removed net N$20: IC3.PB0(ICP), Q6B.B
- removed net N$21: IC3.PD7(AIN1), Q6A.B
- removed net N$22: IC3.PD6(AIN0), Q5B.B
- removed net N$23: IC3.PD5(T1), Q5A.B
- removed net N$24: IC3.PD4(XCK/T0), R16.1
- removed net N$25: IC3.PD3(INT1), R25.1
- removed net N$26: IC3.PC0(ADC0), Q1A.B
- removed net N$27: C3.2, IC3.PB7(XTAL2/TOSC2), Q7.1
- removed net N$28: IC3.PD2(INT0), R26.1
- removed net N$29: IC3.PB4(MISO), R27.1, TP2.TP
- removed net N$36: LED_AM.A, LED_S5.A, U$4.F, U$5.F, U$6.F, U$7.CC
- removed net N$51: LED_AM.C, LED_CW.C, LED_DBG.C, LED_LSB.C, LED_PC.C, LED_S4.A, LED_USB.C, U$4.E, U$5.E, U$6.E, U$7.E
- removed net N$53: LED_DBG.A, LED_S1.C, LED_S2.C, LED_S3.C, LED_S4.C, LED_S5.C, LED_S6.C, LED_S7.C, LED_S8.C, U$4.D, U$5.D, U$6.D, U$7.D
- removed net N$9: LED_S7.A, LED_USB.A, U$4.DP, U$5.CC, U$6.G, U$7.G
- removed net UART_IN: IC3.PD0(RXD), U$2G$6.S
- removed net UART_OUT: IC3.PD1(TXD), U$2G$5.S
- new net BTN_DN: C10.1, R21.2
- new net BTN_RAW_DN: R20.2, R21.1, S_DOWN.1, S_DOWN.2
- new net N$6: D3.C, R6.2, U$10.C, U$11.C, U$9.C
- new net N$77: LED_AM.A, LED_CHG.A, LED_CW.A, LED_DBG.A, LED_LSB.A, LED_PC.A, LED_PWR.A, LED_USB.A
- new net N$82: LED_S2.A, LED_S3.A, LED_S4.A, LED_S5.A, LED_S6.A, LED_S7.A, LED_S8.A, LED_S9.A
- net +3V3: no longer IC3.AREF, IC3.AVCC, IC3.VCC@1, IC3.VCC@2, Q5A.E, Q5B.E, Q6A.E, Q6B.E, Q9A.E, Q9B.E, R10.1, R12.1, R14.1, R24.1, U$2G$1.S, U$2G$2.S
- net BTN_PWR: no longer R16.2
- net BTN_RAW_PWR: now also R22.2, R23.1, S_PWR.1, S_PWR.2; no longer R20.2, R21.1, S_DOWN.1, S_DOWN.2
- net BTN_UP: no longer R25.2
- net GND: no longer C1.2, C2.1, C3.1, C4.2, C5.2, C6.2, IC3.GND, IC3.GND@1, IC3.GND@2, IC3.THERMAL, Q1A.E, Q1B.E, Q2A.E, Q2B.E, Q3A.E, Q3B.E, Q4A.E, Q4B.E, U$2G$7.S, U$2G$8.S, U$3G$4.S
- net N$1: now also D3.DP, R1.2, U$10.DP, U$11.DP, U$9.DP; no longer LED_CW.A, LED_S8.A, U$4.CC, U$5.DP, U$6.DP, U$7.DP
- net N$2: now also D3.G, R2.2, U$10.G, U$11.G, U$9.G; no longer LED_PC.A, LED_S3.A, LED_S9.C, U$4.C, U$5.C, U$6.C, U$7.C
- net N$3: now also D3.F, R3.2, U$10.F, U$11.F, U$9.F; no longer LED_S2.A, LED_S9.A, U$4.B, U$5.B, U$6.B, U$7.B
- net N$4: now also D3.E, R4.2, U$10.E, U$11.E, U$9.E; no longer LED_S1.A, U$4.A, U$5.A, U$6.A, U$7.A
- net N$5: now also D3.D, R5.2, U$10.D, U$11.D, U$9.D; no longer IC3.PC1(ADC1), Q1B.B
- net N$7: now also D3.B, R7.2, U$10.B, U$11.B, U$9.B; no longer IC3.PB5(SCK), R1.1, TP3.TP
- net N$8: now also D3.A, R8.2, U$10.A, U$11.A, U$9.A; no longer IC3.PC2(ADC2), Q2A.B
Other:
- moved on the sheet: C10, C8, C9, LED_AM, LED_CHG, LED_CW, LED_DBG, LED_LSB, LED_PC, LED_PWR, LED_S2, LED_S3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
