File: Hardware/Top.brd (EAGLE design)
At the start: 120 x 80 mm, 44 parts, among them T1 MMBT2222AWT1G, U1 XILINX_DEVICES_6SLX9TQG144, X1 MINI-USB-SCHIELD-32005-201

Commit message: Add various parts
Parts:
- removed U1: XILINX_DEVICES_6SLX9TQG144, MyLib:XILINX_DEVICES_TQ144
- added IC1: MEGA16-M, atmel:MLF44
- added Q1, Q2, Q3, Q4: BC847BS, transistor-small-signal:SOT363_PHILIPS
- added X2: PHB_1MM27_2X08_SNS, _hhn_con_pinhead_box_1mm27:PHB_1MM27_2X08_SNS
- moved U$3 14.3 mm to (67.0, 49.0)
- moved U$4 12.2 mm to (73.0, 49.0)
Connections:
- removed net VCCINT: U1.P128, U1.P19, U1.P28, U1.P52, U1.P89
- new net AVCC: IC1.27
- new net GND1: IC1.18
- new net GND2: IC1.39
- new net VCC1: IC1.17
- new net VCC2: IC1.38
- net +3V3: no longer U1.P103, U1.P122, U1.P125, U1.P129, U1.P135, U1.P18, U1.P20, U1.P31, U1.P36, U1.P4, U1.P42, U1.P53, U1.P63, U1.P76, U1.P86, U1.P90
- net GND: now also IC1.28, IC1.6; no longer U1.P108, U1.P113, U1.P13, U1.P130, U1.P136, U1.P25, U1.P3, U1.P49, U1.P54, U1.P68, U1.P77, U1.P91, U1.P96
- net VCC: now also IC1.5
