File: Hardware/Top.sch (EAGLE design)
At the start: 44 parts, among them T1 MMBT2222AWT1G, U1 XILINX_DEVICES_6SLX9TQG144, X1 MINI-USB-SCHIELD-32005-201

Commit message: Add various parts
Parts:
- removed U1: XILINX_DEVICES_6SLX9TQG144, MyLib:XILINX_DEVICES_6SLX9TQG144
- added IC1: MEGA16-M, atmel:MEGA16-M
- added Q1, Q2, Q3, Q4: BC847BS, transistor-small-signal:BC847BS
- added X2: PHB_1MM27_2X08_SNS, _hhn_con_pinhead_box_1mm27:PHB_1MM27_2X08_SNS
Connections:
- removed net VCCINT: U1BVCCINT.VCCINT@0, U1BVCCINT.VCCINT@1, U1BVCCINT.VCCINT@2, U1BVCCINT.VCCINT@3, U1BVCCINT.VCCINT@4
- net +3V3: no longer U1B0.VCCO_0@0, U1B0.VCCO_0@1, U1B0.VCCO_0@2, U1B1.VCCO_1@0, U1B1.VCCO_1@1, U1B1.VCCO_1@2, U1B2.VCCO_2@0, U1B2.VCCO_2@1, U1B3.VCCO_3@0, U1B3.VCCO_3@1, U1B3.VCCO_3@2, U1BVCCAUX.VCCAUX@0, U1BVCCAUX.VCCAUX@1, U1BVCCAUX.VCCAUX@2, U1BVCCAUX.VCCAUX@3, U1BVCCAUX.VCCAUX@4
- net GND: no longer U1BGND.GND@0, U1BGND.GND@1, U1BGND.GND@10, U1BGND.GND@11, U1BGND.GND@12, U1BGND.GND@2, U1BGND.GND@3, U1BGND.GND@4, U1BGND.GND@5, U1BGND.GND@6, U1BGND.GND@7, U1BGND.GND@8, U1BGND.GND@9
