File: Hardware/Bottom.sch (EAGLE design)
At the start: 105 parts, among them IC1 OP491SOIC_N14, IC2 74AC74D, IC3 74LVC1G17DCK, IC4 LT6231, IC5 SN74CBT3253SOIC16, Q2 25MHz

Commit message: m
Parts:
- C1, C2, C3, C4, C40, C41, C47, C48, C49, C50: device rcl:C-EUC0402 -> rcl:C-EUC0603
- C15, C16, C8, C9: value 10µ -> 4µ7
- C24: device rcl:C-EUC0402 -> rcl:C-EUC0805
- C28: value 1µ -> 4µ7; device rcl:C-EUC0603 -> rcl:C-EUC0805
- C29, C30: value 2µ -> 4µ7
- L3, L4: device rcl:L-EUL3216C -> rcl:L-EUL2012C
- R12, R13: device rcl:R-EU_M0805 -> rcl:R-EU_R0603
- R5, R6: device rcl:R-EU_R0402 -> rcl:R-EU_R0603
Connections:
- removed net N$49: C15.1
- net VDD_DC: now also C15.1

Commit message: Update board Projektarbeit
Parts:
- removed C10, C11, C19, C20: 100n, rcl:C-EUC0603
- removed C6, C7: 22µ, rcl:C-EUC0805
- removed C8, C9: 4µ7, rcl:C-EUC0805
- removed L1: 4.7µH, PowerMagnetics (rev18d):WE-MAPI_3020_74438336047
- removed R1: 54k9, rcl:R-EU_R0603
- removed R2, R6: 10k, rcl:R-EU_R0603
- removed SV3: (no value), con-lstb:MA05-2
- removed U$2: TPS562201, MyLib:TPS562201
- added C43: 22µ, rcl:C-EUC0805
- added D1: (no value), diode:DIODE-SMB
- added TST1, TST2, TST3, TST4: BU-SMA-V, con-coax:BU-SMA-V
- C17, C18: device rcl:C-EUC0603 -> rcl:C-EUC0805
- C5: value 22µ -> 4µ7
- R3, R4, R5: device rcl:R-EU_R0603 -> rcl:R-EU_R0805
Connections:
- removed net +5V: JP1.1, SV3.2, SV3.4
- removed net N$11: R1.2, R2.2, U$2.FB
- removed net N$30: C5.1, C6.1, C7.1, JP1.2, L1.2, R1.1
- removed net N$35: SV4.10
- removed net N$36: SV4.8
- removed net N$37: SV4.6
- removed net N$38: SV4.4
- removed net N$8: C11.2, L1.1, U$2.SW
- removed net RESV_NC: SV4.2
- removed net SPI_MCS_MOSI: SV4.7
- removed net VREG_VDD5_EN: R6.1, U$2.EN
- new net FBPEIHRNG: TST3.1
- new net TST1: TST1.1
- new net TST2: TST2.1
- new net TST4: TST4.1
- new net VCCADC: C30.1, C31.1, JP1.1, L4.1, U$7.DVDD
- net +3V3: now also JP1.2, SV4.10, SV4.8; no longer C19.1, C20.1, C30.1, C31.1, SV3.6, SV3.8, U$7.DVDD
- net ADC_CHSEL: now also SV4.3; no longer SV4.1
- net BASEBAND_I: now also JP3.6; no longer JP3.2
- net BASEBAND_Q: now also JP3.2; no longer JP3.6
- net GND: now also C43.2, SV4.1, SV4.2, TST1.2, TST2.2, TST3.2, TST4.2; no longer C10.2, C19.2, C20.2, C6.2, C7.2, C8.2, C9.2, R2.1, SV3.1, SV3.3, SV3.5, SV3.7, U$2.GND
- net I2C_MCS_SCL: now also SV4.4; no longer SV3.9
- net I2C_MCS_SDA: now also SV4.6; no longer SV3.10
- net N$31: now also C43.1
- net N$7: now also D1.A, J1.3; no longer C11.1, U$2.VBST
- net SPI_MCS_CLK: now also SV4.7; no longer SV4.9
- net SPI_MCS_CS: now also SV4.5; no longer SV4.3
- net SPI_MCS_MISO: now also SV4.9; no longer SV4.5
- net VDD_DC: now also C5.1, D1.C; no longer C10.1, C8.1, C9.1, J1.3, R6.2, U$2.VIN
Other:
- moved on the sheet: C5, JP2, SV4

Commit message: KiCAD advancements
Connections:
- removed net N$23: C34.1, IC5A.1B3, IC5A.2B1, R27.2
- removed net N$53: C33.1, IC5A.1B2, IC5A.2B4, R26.2
- new net N$128: C35.1, IC5A.1B4, IC5A.2B2, R26.2
- new net N$130: C33.1, IC5A.1B2, IC5A.2B4, R27.2
- net N$34: now also C34.1, IC5A.1B3, IC5A.2B1; no longer C35.1, IC5A.1B4, IC5A.2B2
Changed lines of the file:
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@@
-</segment>
-</net>
-<net name="N$23" class="0">
-<segment>
-<pinref part="C34" gate="G$1" pin="1"/>
-<wire x1="182.88" y1="132.08" x2="182.88" y2="137.16" width="0.1524" layer="91"/>
-<wire x1="152.4" y1="137.16" x2="154.94" y2="137.16" width="0.1524" layer="91"/>
-<wire x1="154.94" y1="137.16" x2="182.88" y2="137.16" width="0.1524" layer="91"/>
-<wire x1="152.4" y1="129.54" x2="154.94" y2="129.54" width="0.1524" layer="91"/>
-<wire x1="154.94" y1="129.54" x2="154.94" y2="137.16" width="0.1524" layer="91"/>
-<junction x="154.94" y="137.16"/>
-<wire x1="182.88" y1="137.16" x2="208.28" y2="137.16" width="0.1524" layer="91"/>
-<junction x="182.88" y="137.16"/>
-<wire x1="208.28" y1="137.16" x2="208.28" y2="121.92" width="0.1524" layer="91"/>
-<pinref part="R27" gate="G$1" pin="2"/>
-<wire x1="208.28" y1="121.92" x2="215.9" y2="121.92" width="0.1524" layer="91"/>
-<pinref part="IC5" gate="A" pin="1B3"/>
-<pinref part="IC5" gate="A" pin="2B1"/>
-</segment>
-</net>
-<net name="N$34" class="0">
-<segment>
-<pinref part="C35" gate="G$1" pin="1"/>
-<wire x1="152.4" y1="134.62" x2="157.48" y2="134.62" width="0.1524" layer="91"/>
-<wire x1="157.48" y1="134.62" x2="190.5" y2="134.62" width="0.1524" layer="91"/>
-<wire x1="190.5" y1="132.08" x2="190.5" y2="134.62" width="0.1524" layer="91"/>
-<wire x1="152.4" y1="127" x2="157.48" y2="127" width="0.1524" layer="91"/>
-<wire x1="157.48" y1="127" x2="157.48" y2="134.62" width="0.1524" layer="91"/>
-<junction x="157.48" y="134.62"/>
-<wire x1="190.5" y1="134.62" x2="205.74" y2="134.62" width="0.1524" layer="91"/>
-<junction x="190.5" y="134.62"/>
-<wire x1="205.74" y1="134.62" x2="205.74" y2="116.84" width="0.1524" layer="91"/>
-<pinref part="R28" gate="G$1" pin="2"/>
-<wire x1="205.74" y1="116.84" x2="215.9" y2="116.84" width="0.1524" layer="91"/>
-<pinref part="IC5" gate="A" pin="1B4"/>
-<pinref part="IC5" gate="A" pin="2B2"/>
-</segment>
-</net>
-<net name="N$53" class="0">
-<segment>
-<pinref part="C33" gate="G$1" pin="1"/>
-<wire x1="152.4" y1="139.7" x2="162.56" y2="139.7" width="0.1524" layer="91"/>
-<wire x1="162.56" y1="139.7" x2="175.26" y2="139.7" width="0.1524" layer="91"/>
-<wire x1="175.26" y1="132.08" x2="175.26" y2="139.7" width="0.1524" layer="91"/>
-<wire x1="152.4" y1="121.92" x2="162.56" y2="121.92" width="0.1524" layer="91"/>
-<wire x1="162.56" y1="121.92" x2="162.56" y2="139.7" width="0.1524" layer="91"/>
-<junction x="162.56" y="139.7"/>
-<wire x1="175.26" y1="139.7" x2="210.82" y2="139.7" width="0.1524" layer="91"/>
-<junction x="175.26" y="139.7"/>
-<wire x1="210.82" y1="139.7" x2="210.82" y2="137.16" width="0.1524" layer="91"/>
-<pinref part="R26" gate="G$1" pin="2"/>
-<wire x1="210.82" y1="137.16" x2="215.9" y2="137.16" width="0.1524" layer="91"/>
-<pinref part="IC5" gate="A" pin="1B2"/>
-<pinref part="IC5" gate="A" pin="2B4"/>
 </segment>
 </net>
@@
 </segment>
 </net>
+<net name="N$128" class="0">
+<segment>
+<pinref part="C35" gate="G$1" pin="1"/>
+<wire x1="152.4" y1="134.62" x2="157.48" y2="134.62" width="0.1524" layer="91"/>
+<wire x1="157.48" y1="134.62" x2="190.5" y2="134.62" width="0.1524" layer="91"/>
+<wire x1="190.5" y1="132.08" x2="190.5" y2="134.62" width="0.1524" layer="91"/>
+<wire x1="152.4" y1="127" x2="157.48" y2="127" width="0.1524" layer="91"/>
+<wire x1="157.48" y1="127" x2="157.48" y2="134.62" width="0.1524" layer="91"/>
+<junction x="157.48" y="134.62"/>
+<pinref part="IC5" gate="A" pin="1B4"/>
+<pinref part="IC5" gate="A" pin="2B2"/>
+<wire x1="190.5" y1="134.62" x2="213.36" y2="134.62" width="0.1524" layer="91"/>
+<junction x="190.5" y="134.62"/>
+<wire x1="213.36" y1="134.62" x2="213.36" y2="137.16" width="0.1524" layer="91"/>
+<pinref part="R26" gate="G$1" pin="2"/>
+<wire x1="213.36" y1="137.16" x2="215.9" y2="137.16" width="0.1524" layer="91"/>
+</segment>
+</net>
+<net name="N$130" class="0">
+<segment>
+<pinref part="C33" gate="G$1" pin="1"/>
+<wire x1="152.4" y1="139.7" x2="162.56" y2="139.7" width="0.1524" layer="91"/>
+<wire x1="162.56" y1="139.7" x2="175.26" y2="139.7" width="0.1524" layer="91"/>
+<wire x1="175.26" y1="132.08" x2="175.26" y2="139.7" width="0.1524" layer="91"/>
+<wire x1="152.4" y1="121.92" x2="162.56" y2="121.92" width="0.1524" layer="91"/>
+<wire x1="162.56" y1="121.92" x2="162.56" y2="139.7" width="0.1524" layer="91"/>
+<junction x="162.56" y="139.7"/>
+<pinref part="IC5" gate="A" pin="1B2"/>
+<pinref part="IC5" gate="A" pin="2B4"/>
+<wire x1="208.28" y1="139.7" x2="175.26" y2="139.7" width="0.1524" layer="91"/>
+<junction x="175.26" y="139.7"/>
+<pinref part="R27" gate="G$1" pin="2"/>
+<wire x1="208.28" y1="121.92" x2="215.9" y2="121.92" width="0.1524" layer="91"/>
+<wire x1="208.28" y1="139.7" x2="208.28" y2="121.92" width="0.1524" layer="91"/>
+</segment>
+</net>
+<net name="N$34" class="0">
+<segment>
+<pinref part="R28" gate="G$1" pin="2"/>
+<wire x1="205.74" y1="116.84" x2="215.9" y2="116.84" width="0.1524" layer="91"/>
+<wire x1="205.74" y1="116.84" x2="205.74" y2="137.16" width="0.1524" layer="91"/>
+<pinref part="C34" gate="G$1" pin="1"/>
+<wire x1="182.88" y1="132.08" x2="182.88" y2="137.16" width="0.1524" layer="91"/>
+<wire x1="152.4" y1="137.16" x2="154.94" y2="137.16" width="0.1524" layer="91"/>
+<wire x1="154.94" y1="137.16" x2="182.88" y2="137.16" width="0.1524" layer="91"/>
+<wire x1="152.4" y1="129.54" x2="154.94" y2="129.54" width="0.1524" layer="91"/>
+<wire x1="154.94" y1="129.54" x2="154.94" y2="137.16" width="0.1524" layer="91"/>
+<junction x="154.94" y="137.16"/>
+<pinref part="IC5" gate="A" pin="1B3"/>
+<pinref part="IC5" gate="A" pin="2B1"/>
+<wire x1="205.74" y1="137.16" x2="182.88" y2="137.16" width="0.1524" layer="91"/>
+<junction x="182.88" y="137.16"/>
+</segment>
+</net>
