File: Hardware/Bottom/GeckoTRX_Bottom.kicad_pcb (KiCad board)
At the start: 2 copper layers, 120 x 80 mm, 192 parts, among them J1 Jack-DC, J2 Conn_Coaxial, J3 Conn_02x05_Odd_Even, J4 Conn_02x05_Odd_Even, K1 G6K-2, K2 G6K-2, K3 G6K-2, K4 G6K-2, T1 Transformer_1P_SS, U1 TPS562200, U2 SN74CBT3253, U3 OP249, U4 ADA4807-4, U5 MCP23017_ML, U6 Si5351A-B-GM, U7 LM79M12_TO220, U8 LM79M12_TO220, Y1 25MHz

Commit message: KiCAD advancements
Parts:
- removed U7, U8: LM79M12_TO220, Package_TO_SOT_THT:TO-220-3_Horizontal_TabDown
- added C99: 1u, Capacitor_SMD:C_0805_2012Metric, F.Cu at (-28.0, 24.0)
- moved C17 18.0 mm to (2.00, 31.0), turned to 180 degrees
- moved C24 17.7 mm to (-28.0, 28.0), turned to 270 degrees
- moved C20 16.1 mm to (2.00, 29.0), turned to 180 degrees
- moved R11 14.6 mm to (2.00, 27.0), turned to 0 degrees
- moved C32 11.0 mm to (-0.89, 6.59)
- moved C33 11.0 mm to (-0.89, 8.59)
- moved C34 11.0 mm to (-0.89, 13.1)
- moved C35 11.0 mm to (-0.89, 15.1)
- moved C36 11.0 mm to (-10.9, 16.1)
- moved C37 11.0 mm to (-10.9, 14.1)
- moved C38 11.0 mm to (-7.89, 7.09)
- moved R24 11.0 mm to (-10.9, 10.1)
- moved R25 11.0 mm to (-10.9, 8.09)
- moved R26 11.0 mm to (-10.9, 6.09)
- moved U6 11.0 mm to (-5.89, 12.1)
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Connections:
- C75 pad 2: /Bandfilter/LPF_80M_OUT -> /Bandfilter/LPF_80M_IN
- C76 pad 2: /Bandfilter/LPF_40M_OUT -> /Bandfilter/LPF_40M_IN
- C77 pad 2: /Bandfilter/LPF_20M_OUT -> /Bandfilter/LPF_20M_IN
- C78 pad 2: /Bandfilter/LPF_80M_OUT -> /Bandfilter/LPF_80M_IN
- C79 pad 2: /Bandfilter/LPF_40M_OUT -> /Bandfilter/LPF_40M_IN
- C80 pad 2: /Bandfilter/LPF_20M_OUT -> /Bandfilter/LPF_20M_IN
- C93 pad 2: /Bandfilter/LPF_80M_IN -> /Bandfilter/LPF_80M_OUT
- C94 pad 2: /Bandfilter/LPF_40M_IN -> /Bandfilter/LPF_40M_OUT
- C95 pad 2: /Bandfilter/LPF_20M_IN -> /Bandfilter/LPF_20M_OUT
- C96 pad 2: /Bandfilter/LPF_80M_IN -> /Bandfilter/LPF_80M_OUT
- C97 pad 2: /Bandfilter/LPF_40M_IN -> /Bandfilter/LPF_40M_OUT
- C98 pad 2: /Bandfilter/LPF_20M_IN -> /Bandfilter/LPF_20M_OUT
- K1 pad 3: /Bandfilter/LPF_80M_OUT -> /Bandfilter/LPF_80M_IN
- K1 pad 4: /Bandfilter/LPF_OUT -> /Bandfilter/LPF_IN
- K1 pad 5: /Bandfilter/LPF_IN -> /Bandfilter/LPF_OUT
- K1 pad 6: /Bandfilter/LPF_80M_IN -> /Bandfilter/LPF_80M_OUT
- K2 pad 3: /Bandfilter/LPF_40M_OUT -> /Bandfilter/LPF_40M_IN
- K2 pad 4: /Bandfilter/LPF_OUT -> /Bandfilter/LPF_IN
- K2 pad 5: /Bandfilter/LPF_IN -> /Bandfilter/LPF_OUT
- K2 pad 6: /Bandfilter/LPF_40M_IN -> /Bandfilter/LPF_40M_OUT
- K3 pad 3: /Bandfilter/LPF_20M_OUT -> /Bandfilter/LPF_20M_IN
- K3 pad 4: /Bandfilter/LPF_OUT -> /Bandfilter/LPF_IN
- K3 pad 5: /Bandfilter/LPF_IN -> /Bandfilter/LPF_OUT
- K3 pad 6: /Bandfilter/LPF_20M_IN -> /Bandfilter/LPF_20M_OUT
- L18 pad 1: /Bandfilter/LPF_80M_OUT -> /Bandfilter/LPF_80M_IN
- L19 pad 1: /Bandfilter/LPF_40M_OUT -> /Bandfilter/LPF_40M_IN
- L20 pad 1: /Bandfilter/LPF_20M_OUT -> /Bandfilter/LPF_20M_IN
- L24 pad 2: /Bandfilter/LPF_80M_IN -> /Bandfilter/LPF_80M_OUT
- L25 pad 2: /Bandfilter/LPF_40M_IN -> /Bandfilter/LPF_40M_OUT
- L26 pad 2: /Bandfilter/LPF_20M_IN -> /Bandfilter/LPF_20M_OUT
Other:
- outline, holes or cut-outs redrawn

Commit message: KiCAD advancements
Parts:
- removed R4, R5, R6, R7: 100R, Resistor_SMD:R_0805_2012Metric
- added C100: 10n, Capacitor_SMD:C_0805_2012Metric, F.Cu at (-20.0, 28.0)
- moved C6 16.6 mm to (-20.0, 24.0), turned to 90 degrees
- moved C9 11.1 mm to (-16.5, 20.5)
- moved C12 8.28 mm to (-16.5, 31.5)
- moved T1 7.76 mm to (-3.50, 23.0)
- moved C17 7.50 mm to (-5.50, 31.0)
- moved C20 7.50 mm to (-5.50, 29.0)
- moved C21 7.50 mm to (-1.50, 27.0)
- moved L2 7.50 mm to (-1.50, 31.0)
- moved R11 7.50 mm to (-5.50, 27.0)
- moved R8 7.50 mm to (-1.50, 29.0)
- moved U2 7.50 mm to (-13.5, 26.0), turned to 90 degrees
- moved C8 4.30 mm to (-10.5, 31.5), turned to 0 degrees
- moved C38 4.00 mm to (-11.9, 7.09)
- moved U6 4.00 mm to (-9.89, 12.1)
- moved Y1 4.00 mm to (-8.39, 7.09)
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Connections:
- R10 pad 2: Net-(R10-Pad2) -> Net-(C10-Pad1)
- R9 pad 1: Net-(R5-Pad2) -> Net-(C12-Pad1)
- U3 pad 2: Net-(R5-Pad2) -> Net-(C12-Pad1)
- U3 pad 3: Net-(R4-Pad2) -> Net-(C8-Pad1)
- U3 pad 5: Net-(R6-Pad2) -> Net-(C9-Pad1)
- U3 pad 6: Net-(R10-Pad2) -> Net-(C10-Pad1)
Routing:
- net Net-(C12-Pad1): track 0.00 -> 11.0 mm, vias 0 -> 2
- net Net-(C10-Pad1): track 0.00 -> 11.0 mm, vias 0 -> 3
- net Net-(C8-Pad1): track 0.00 -> 5.93 mm
- net Net-(C9-Pad1): track 0.00 -> 5.93 mm
- net (no net): vias 5 -> 24

Commit message: Update
Parts:
- removed C100: 10n, Capacitor_SMD:C_0805_2012Metric
- removed C47, C49, C51, C53, C54, C55, C56, C57, C58, C59, C61, C63, C65, C66, C67, C68, C69, C70, C71, C72, C73, C74, C75, C76, C77, C78, C79, C80, C81, C82, C83, C84, C85, C86, C87, C88, C89, C90, C91, C92, C93, C94, C95, C96, C97, C98: 68p, Capacitor_SMD:C_0805_2012Metric
- removed C48, C50, C52, C60, C62, C64: C_Variable, Capacitor_SMD:C_Trimmer_Murata_TZB4-B
- removed C99: 1u, Capacitor_SMD:C_0805_2012Metric
- removed D10, D11, D6, D7, D8, D9: D, Package_TO_SOT_SMD:SOT-23
- removed K1, K2, K3: G6K-2, Relay_SMD:Relay_DPDT_Omron_G6K-2G-Y
- removed L10, L11, L12, L13, L14, L18, L19, L20, L21, L22, L23, L24, L25, L26, L9: L, Inductor_SMD:L_1812_4532Metric
- removed L15, L16, L17, L3, L4, L5, L6, L7, L8: L_Core_Ferrite, Inductor_SMD:L_1812_4532Metric
- removed R30, R31, R32, R33, R34, R35: 100R, Resistor_SMD:R_0805_2012Metric
- added IPHOUT1: Conn_Coaxial, Connector_Coaxial:SMA_Amphenol_132134-11_Vertical, F.Cu at (-45.0, 26.0)
- added J10: Conn_01x04_Female, Connector_PinSocket_1.27mm:PinSocket_1x04_P1.27mm_Vertical_SMD_Pin1Left, F.Cu at (27.0, 15.0)
- added J11: Conn_01x04_Female, Connector_PinSocket_1.27mm:PinSocket_1x04_P1.27mm_Vertical_SMD_Pin1Left, F.Cu at (27.0, 22.0)
- added J12: Conn_01x03_Female, Connector_PinSocket_1.27mm:PinSocket_1x03_P1.27mm_Vertical_SMD_Pin1Left, F.Cu at (49.0, -20.0)
- added J13: Conn_01x03_Female, Connector_PinSocket_1.27mm:PinSocket_1x03_P1.27mm_Vertical_SMD_Pin1Left, F.Cu at (49.0, -13.0)
- added J14: Conn_01x03_Female, Connector_PinSocket_1.27mm:PinSocket_1x03_P1.27mm_Vertical_SMD_Pin1Left, F.Cu at (49.0, -6.00)
- added J15: Conn_01x03_Female, Connector_PinSocket_1.27mm:PinSocket_1x03_P1.27mm_Vertical_SMD_Pin1Left, F.Cu at (49.0, 1.00)
- added J16: Conn_01x03_Female, Connector_PinSocket_1.27mm:PinSocket_1x03_P1.27mm_Vertical_SMD_Pin1Left, F.Cu at (49.0, 8.00)
- added J17: Conn_01x03_Female, Connector_PinSocket_1.27mm:PinSocket_1x03_P1.27mm_Vertical_SMD_Pin1Left, F.Cu at (49.0, 15.0)
- added J18: Conn_01x03_Female, Connector_PinSocket_1.27mm:PinSocket_1x03_P1.27mm_Vertical_SMD_Pin1Left, F.Cu at (49.0, 22.0)
- added J19: Conn_01x03_Female, Connector_PinSocket_1.27mm:PinSocket_1x03_P1.27mm_Vertical_SMD_Pin1Left, F.Cu at (-30.0, -12.0)
- added J20: Conn_01x03_Female, Connector_PinSocket_1.27mm:PinSocket_1x03_P1.27mm_Vertical_SMD_Pin1Left, F.Cu at (-23.0, -12.0)
- added J21: Conn_01x03_Female, Connector_PinSocket_1.27mm:PinSocket_1x03_P1.27mm_Vertical_SMD_Pin1Left, F.Cu at (-16.0, -12.0)
- added J22: Conn_01x03_Female, Connector_PinSocket_1.27mm:PinSocket_1x03_P1.27mm_Vertical_SMD_Pin1Left, F.Cu at (-9.00, -12.0)
- added J23: Conn_01x03_Female, Connector_PinSocket_1.27mm:PinSocket_1x03_P1.27mm_Vertical_SMD_Pin1Left, F.Cu at (-2.00, -12.0)
- added J24: Conn_01x03_Female, Connector_PinSocket_1.27mm:PinSocket_1x03_P1.27mm_Vertical_SMD_Pin1Left, F.Cu at (5.00, -12.0)
- added J25: Conn_01x03_Female, Connector_PinSocket_1.27mm:PinSocket_1x03_P1.27mm_Vertical_SMD_Pin1Left, F.Cu at (12.0, -12.0)
- added J26: Conn_01x03_Female, Connector_PinSocket_1.27mm:PinSocket_1x03_P1.27mm_Vertical_SMD_Pin1Left, F.Cu at (-30.0, -34.0)
- added J27: Conn_01x03_Female, Connector_PinSocket_1.27mm:PinSocket_1x03_P1.27mm_Vertical_SMD_Pin1Left, F.Cu at (-23.0, -34.0)
- added J28: Conn_01x03_Female, Connector_PinSocket_1.27mm:PinSocket_1x03_P1.27mm_Vertical_SMD_Pin1Left, F.Cu at (-16.0, -34.0)
- added J29: Conn_01x03_Female, Connector_PinSocket_1.27mm:PinSocket_1x03_P1.27mm_Vertical_SMD_Pin1Left, F.Cu at (-9.00, -34.0)
- added J30: Conn_01x03_Female, Connector_PinSocket_1.27mm:PinSocket_1x03_P1.27mm_Vertical_SMD_Pin1Left, F.Cu at (-2.00, -34.0)
- added J31: Conn_01x03_Female, Connector_PinSocket_1.27mm:PinSocket_1x03_P1.27mm_Vertical_SMD_Pin1Left, F.Cu at (5.00, -34.0)
- added J32: Conn_01x03_Female, Connector_PinSocket_1.27mm:PinSocket_1x03_P1.27mm_Vertical_SMD_Pin1Left, F.Cu at (12.0, -34.0)
- added J5: Conn_01x04_Female, Connector_PinSocket_1.27mm:PinSocket_1x04_P1.27mm_Vertical_SMD_Pin1Left, F.Cu at (27.0, -20.0)
- added J6: Conn_01x04_Female, Connector_PinSocket_1.27mm:PinSocket_1x04_P1.27mm_Vertical_SMD_Pin1Left, F.Cu at (27.0, -13.0)
- added J7: Conn_01x04_Female, Connector_PinSocket_1.27mm:PinSocket_1x04_P1.27mm_Vertical_SMD_Pin1Left, F.Cu at (27.0, -6.00)
- added J8: Conn_01x04_Female, Connector_PinSocket_1.27mm:PinSocket_1x04_P1.27mm_Vertical_SMD_Pin1Left, F.Cu at (27.0, 1.00)
- added J9: Conn_01x04_Female, Connector_PinSocket_1.27mm:PinSocket_1x04_P1.27mm_Vertical_SMD_Pin1Left, F.Cu at (27.0, 8.00)
- added LO1: Conn_Coaxial, Connector_Coaxial:SMA_Amphenol_132134-11_Vertical, F.Cu at (18.0, 2.00)
- added QPHOUT1: Conn_Coaxial, Connector_Coaxial:SMA_Amphenol_132134-11_Vertical, F.Cu at (-42.0, 18.0)
- added R4: 100R, Resistor_SMD:R_0805_2012Metric, F.Cu at (-13.0, 27.0)
- added R5: 100R, Resistor_SMD:R_0805_2012Metric, F.Cu at (-13.0, 31.0)
- added R6: 100R, Resistor_SMD:R_0805_2012Metric, F.Cu at (-13.0, 19.0)
- added R7: 100R, Resistor_SMD:R_0805_2012Metric, F.Cu at (-13.0, 23.0)
- added RF1: Conn_Coaxial, Connector_Coaxial:SMA_Amphenol_132134-11_Vertical, F.Cu at (-82.0, -21.0)
- added TP1: TestPoint, TestPoint:TestPoint_Pad_D1.0mm, F.Cu at (12.0, 0.00)
- added U10: 74LVC1G17, Package_TO_SOT_SMD:SOT-353_SC-70-5, F.Cu at (9.00, 0.00)
- added U11: 74HC74D, Package_SO:SOIC-14_3.9x8.7mm_P1.27mm, F.Cu at (1.50, 1.50)
- added U7: LM79M12_TO220, Package_TO_SOT_THT:TO-220-3_Horizontal_TabDown, F.Cu at (-12.0, -60.0)
- added U8: LM79M12_TO220, Package_TO_SOT_THT:TO-220-3_Horizontal_TabDown, F.Cu at (-5.00, -65.0)
- added U9: MCP23017_ML, Package_DFN_QFN:QFN-28-1EP_6x6mm_P0.65mm_EP4.25x4.25mm, F.Cu at (-39.0, -4.00)
- C11: value 4u7 -> 1u
- C13: value 4u7 -> 100n
- C39, C40, C41, C42: value 68p -> 100n
- C43: value 68p -> 10n
- C44, C45: value 68p -> 330u; footprint Capacitor_SMD:C_0805_2012Metric -> Capacitor_SMD:C_Elec_6.3x7.7
- C46: value 68p -> DNP
- R27, R28: value 100R -> 10k
- R29: value 100R -> DNP
- U3: value OP249 -> LT6231
- U4: value ADA4807-4 -> OP491-4
- moved C44 95.7 mm to (-50.0, -7.00), turned to 180 degrees
- moved C45 88.7 mm to (-39.0, -15.0), turned to 90 degrees
- moved C46 37.1 mm to (17.0, 20.0), turned to 0 degrees
- moved C42 35.0 mm to (-0.50, -4.50), turned to 180 degrees
- moved C40 34.3 mm to (12.0, 3.50), turned to 270 degrees
- moved C41 31.8 mm to (9.50, -3.50), turned to 270 degrees
- moved C39 30.5 mm to (7.00, -3.50)
- moved R29 27.0 mm to (12.0, -3.50)
- moved C17 25.5 mm to (20.0, 31.0), turned to 270 degrees
- moved R27 25.4 mm to (7.00, 3.50), turned to 90 degrees
- moved C43 25.1 mm to (3.50, -4.50), turned to 180 degrees
- moved C11 25.1 mm to (-31.0, 10.0)
- moved C20 23.6 mm to (18.0, 31.0), turned to 270 degrees
- moved C30 23.1 mm to (-29.0, 9.42)
- moved C31 23.1 mm to (-27.0, 9.42)
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Connections:
- net BB_IPH renamed Net-(C28-Pad1)
- net BB_QPH renamed Net-(C29-Pad2)
- C13 pad 1: +3V3 -> GND
- C13 pad 2: GND -> +3V3
- C39 pad 1: GND -> +3V3
- C39 pad 2: Net-(C39-Pad2) -> GND
- C40 pad 1: GND -> Net-(C40-Pad1)
- C41 pad 2: Net-(C41-Pad2) -> +3V3
- C42 pad 1: Net-(C42-Pad1) -> +3V3
- C42 pad 2: Net-(C42-Pad2) -> GND
- C43 pad 2: Net-(C42-Pad1) -> +3V3
- C44 pad 1: Net-(C44-Pad1) -> +3V3
- C44 pad 2: Net-(C44-Pad2) -> GND
- C45 pad 1: GND -> +3V3
- C45 pad 2: Net-(C44-Pad1) -> GND
- K4 pad 3: /Bandfilter/PRE_IN -> /Filter/SIG_PRE_IN
- K4 pad 6: /Bandfilter/LPF_OUT -> /Filter/SIG_LP_OUT
- R10 pad 2: Net-(C10-Pad1) -> Net-(R10-Pad2)
- R27 pad 1: Net-(C55-Pad2) -> Net-(C40-Pad1)
- R27 pad 2: GND -> +3V3
- R28 pad 1: Net-(C57-Pad2) -> GND
- R28 pad 2: GND -> Net-(C40-Pad1)
- R29 pad 1: Net-(C59-Pad2) -> GND
- R29 pad 2: GND -> Net-(C40-Pad1)
- R9 pad 1: Net-(C12-Pad1) -> Net-(R5-Pad2)
- T1 pad 1: Net-(T1-Pad1) -> Net-(C46-Pad2)
- U2 pad 10: Net-(C10-Pad1) -> Net-(C12-Pad1)
- U2 pad 11: Net-(C12-Pad1) -> Net-(C10-Pad1)
- U2 pad 12: Net-(C8-Pad1) -> Net-(C9-Pad1)
- U2 pad 13: Net-(C9-Pad1) -> Net-(C8-Pad1)
- U3 pad 2: Net-(C12-Pad1) -> Net-(R5-Pad2)
- U3 pad 3: Net-(C8-Pad1) -> Net-(R4-Pad2)
- U3 pad 5: Net-(C9-Pad1) -> Net-(R6-Pad2)
- U3 pad 6: Net-(C10-Pad1) -> Net-(R10-Pad2)
Routing:
- net Net-(C10-Pad1): track 11.0 -> 8.82 mm, vias 3 -> 2
- net Net-(C9-Pad1): track 5.93 -> 7.59 mm
- net Net-(C8-Pad1): track 5.93 -> 7.39 mm, vias 0 -> 2
- net Net-(C12-Pad1): track 11.0 -> 9.92 mm
- net GND: vias 4 -> 3
- net (no net): vias 24 -> 3
Other:
- outline, holes or cut-outs redrawn

Commit message: Update
Parts:
- removed IPHOUT1, QPHOUT1: Conn_Coaxial, Connector_Coaxial:SMA_Amphenol_132134-11_Vertical
- removed U8: LM79M12_TO220, Package_TO_SOT_THT:TO-220-3_Horizontal_TabDown
- removed U9: MCP23017_ML, Package_DFN_QFN:QFN-28-1EP_6x6mm_P0.65mm_EP4.25x4.25mm
- added C47: 100n, Capacitor_SMD:C_0805_2012Metric, F.Cu at (0.07, 30.2)
- added C48: 100n, Capacitor_SMD:C_0805_2012Metric, F.Cu at (-17.6, 70.3)
- added C49: 100n, Capacitor_SMD:C_0805_2012Metric, F.Cu at (-17.6, 72.3)
- added C50: 10p, Capacitor_SMD:C_0805_2012Metric, F.Cu at (14.0, 9.00)
- added C51: 10p, Capacitor_SMD:C_0805_2012Metric, F.Cu at (19.0, 9.00)
- added C52: 1u, Capacitor_SMD:C_0805_2012Metric, F.Cu at (-27.0, 65.0)
- added C53: 100n, Capacitor_SMD:C_0805_2012Metric, F.Cu at (-27.0, 68.0)
- added C54: 15n, Capacitor_SMD:C_0805_2012Metric, F.Cu at (-14.0, 12.0)
- added IOUT1: Conn_Coaxial, Connector_Coaxial:SMA_Amphenol_132134-11_Vertical, F.Cu at (-41.0, 29.0)
- added QOUT1: Conn_Coaxial, Connector_Coaxial:SMA_Amphenol_132134-11_Vertical, F.Cu at (-41.0, 19.0)
- added R30: 0R, Resistor_SMD:R_0805_2012Metric, F.Cu at (-15.5, 51.9)
- added R31: 0R, Resistor_SMD:R_0805_2012Metric, F.Cu at (-12.1, 49.9)
- added R32: 10, Resistor_SMD:R_0805_2012Metric, F.Cu at (18.0, -24.0)
- added R33: 10, Resistor_SMD:R_0805_2012Metric, F.Cu at (20.0, -24.0)
- added R34: 0R, Resistor_SMD:R_0805_2012Metric, F.Cu at (-12.1, 48.0)
- added R35: 0R, Resistor_SMD:R_0805_2012Metric, F.Cu at (4.00, 9.00)
- added R36: 0R, Resistor_SMD:R_0805_2012Metric, F.Cu at (-7.00, 0.50)
- added R37: 0R, Resistor_SMD:R_0805_2012Metric, F.Cu at (-7.00, 3.00)
- added R38: DNP, Resistor_SMD:R_0805_2012Metric, F.Cu at (21.0, 25.0)
- added R39: 1k, Resistor_SMD:R_0805_2012Metric, F.Cu at (14.0, 7.00)
- added R40: 1k, Resistor_SMD:R_0805_2012Metric, F.Cu at (8.00, 8.00)
- added R41: 10k, Resistor_SMD:R_0805_2012Metric, F.Cu at (-27.0, 62.0)
- added R42: 50, Resistor_SMD:R_1206_3216Metric, F.Cu at (-51.0, -5.00)
- added R43: 0R, Resistor_SMD:R_0402_1005Metric, F.Cu at (-53.0, -4.00)
- added R44: 50, Resistor_SMD:R_1206_3216Metric, F.Cu at (-45.0, -5.00)
- added R45: 50, Resistor_SMD:R_1206_3216Metric, F.Cu at (-48.0, -5.00)
- added R46: 10, Resistor_SMD:R_0805_2012Metric, F.Cu at (-11.5, 6.50)
- added R47: 10, Resistor_SMD:R_0805_2012Metric, F.Cu at (-9.00, 6.50)
- added RV1: 100, Potentiometer_SMD:Potentiometer_Bourns_3224W_Vertical, F.Cu at (-17.0, 31.0)
- added RV2: 100, Potentiometer_SMD:Potentiometer_Bourns_3224W_Vertical, F.Cu at (-18.0, 13.0)
- added RV3: R_POT, Potentiometer_SMD:Potentiometer_Bourns_3224W_Vertical, F.Cu at (18.0, 47.0)
- added TP10: 180, TestPoint:TestPoint_Pad_D1.0mm, F.Cu at (10.0, 22.0)
- added TP11: GND, TestPoint:TestPoint_Pad_D1.0mm, F.Cu at (16.0, 37.0)
- added TP12: TestPoint, TestPoint:TestPoint_Pad_D1.0mm, F.Cu at (-18.0, 43.0)
- added TP13: TestPoint, TestPoint:TestPoint_Pad_D1.0mm, F.Cu at (-19.6, 55.8)
- added TP14: TestPoint, TestPoint:TestPoint_Pad_D1.0mm, F.Cu at (-15.5, 56.0)
- added TP15: TestPoint, TestPoint:TestPoint_Pad_D1.0mm, F.Cu at (-11.0, 53.0)
- added TP18: TestPoint, TestPoint:TestPoint_Pad_D1.0mm, F.Cu at (14.0, 8.00)
- added TP19: TestPoint, TestPoint:TestPoint_Pad_D1.0mm, F.Cu at (19.6, 5.03)
- added TP2: RFin, TestPoint:TestPoint_Pad_D1.0mm, F.Cu at (16.0, 25.0)
- added TP20: 1V65, TestPoint:TestPoint_Pad_D1.0mm, F.Cu at (4.07, 25.2)
- added TP3: RFp, TestPoint:TestPoint_Pad_D1.0mm, F.Cu at (1.07, 26.2)
- added TP4: RFn, TestPoint:TestPoint_Pad_D1.0mm, F.Cu at (7.07, 26.2)
- added TP5: CLKI, TestPoint:TestPoint_Pad_D1.0mm, F.Cu at (-11.4, 56.2)
- added TP6: CLKQ, TestPoint:TestPoint_Pad_D1.0mm, F.Cu at (-48.0, 47.0)
- added TP7: 000, TestPoint:TestPoint_Pad_D1.0mm, F.Cu at (10.0, 16.0)
- added TP8: 090, TestPoint:TestPoint_Pad_D1.0mm, F.Cu at (10.0, 18.0)
- added TP9: 270, TestPoint:TestPoint_Pad_D1.0mm, F.Cu at (10.0, 20.0)
- added TPI1: TestPoint, TestPoint:TestPoint_Pad_D1.0mm, F.Cu at (1.03, 63.4)
- added TPQ1: TestPoint, TestPoint:TestPoint_Pad_D1.0mm, F.Cu at (3.08, 63.4)
- C1, C24, C25: value 100n -> 10n
- C13: value 100n -> 1u
- C16, C17, C2, C3, C4: value 4u7 -> 10u
- C46: value DNP -> 15n
- R10, R20, R21, R22, R23, R4, R5, R6, R7, R9: value 100R -> 100
- R11: value 10k -> 2k
- R25, R26: value 10k -> DNP
- R8: value 10k -> 1k
- T1: value Transformer_1P_SS -> MABA-007237-ETC410
- U2: value SN74CBT3253 -> SN74CBTLV3253
- U7: value LM79M12_TO220 -> MCP23017_ML; footprint Package_TO_SOT_THT:TO-220-3_Horizontal_TabDown -> Package_DFN_QFN:QFN-28-1EP_6x6mm_P0.65mm_EP4.25x4.25mm
- moved RF1 107.7 mm to (18.0, 19.0)
- moved J12 80.2 mm to (-30.0, -34.0), turned to 180 degrees
- moved J26 80.2 mm to (49.0, -20.0), turned to 90 degrees
- moved J13 75.0 mm to (-23.0, -34.0), turned to 180 degrees
- moved J27 75.0 mm to (49.0, -13.0), turned to 90 degrees
- moved U7 71.9 mm to (-38.0, 7.00), turned to 0 degrees
- moved J14 70.8 mm to (-16.0, -34.0), turned to 180 degrees
- moved J28 70.8 mm to (49.0, -6.00), turned to 90 degrees
- moved J15 67.7 mm to (-9.00, -34.0), turned to 180 degrees
- moved J29 67.7 mm to (49.0, 1.00), turned to 90 degrees
- moved J18 67.1 mm to (12.0, -34.0), turned to 180 degrees
- moved J32 67.1 mm to (49.0, 22.0), turned to 90 degrees
- moved J16 66.1 mm to (-2.00, -34.0), turned to 180 degrees
- moved J30 66.1 mm to (49.0, 8.00), turned to 90 degrees
- moved J17 65.9 mm to (5.00, -34.0), turned to 180 degrees
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Connections:
- net /Filter/SIG_PA_OUT renamed /Filter/SIG_LP_IN
- net /Filter/SW_LP_COM renamed /Filter/REL_COM
- net /Filter/SW_LP_CUSTOM renamed /Filter/SW_LP_CUST
- net /Filter/SW_PRE_10 renamed /Filter/EN_PRE_10
- net /Filter/SW_PRE_15 renamed /Filter/EN_PRE_15
- net /Filter/SW_PRE_160 renamed /Filter/EN_PRE_160
- net /Filter/SW_PRE_20 renamed /Filter/EN_PRE_20
- net /Filter/SW_PRE_40 renamed /Filter/EN_PRE_40
- net /Filter/SW_PRE_80 renamed /Filter/EN_PRE_80
- net /Filter/SW_PRE_CUSTOM renamed /Filter/EN_PRE_CUS
- net /Local oscillator/LO_TST_RX renamed /Filter/LO_TEST_RX
- net Net-(U7-Pad1) renamed /GPIO Expander/GPIO_4
- net Net-(U7-Pad2) renamed /GPIO Expander/GPIO_5
- net Net-(U7-Pad3) renamed /GPIO Expander/GPIO_6
- C1 pad 1: Net-(C1-Pad1) -> +3V3
- C1 pad 2: Net-(C1-Pad2) -> GND
- C13 pad 1: GND -> +3V3
- C13 pad 2: +3V3 -> GND
- C16 pad 1: /Power Supply/1V65 -> Net-(C16-Pad1)
- C17 pad 1: /Power Supply/1V65 -> Net-(C16-Pad1)
- C20 pad 1: /Power Supply/1V65 -> Net-(C16-Pad1)
- C21 pad 1: /Power Supply/1V65 -> 1V65
- C36 pad 1: +3V3 -> Net-(C36-Pad1)
- C36 pad 2: GND -> Net-(C36-Pad2)
- J2 pad 2: Net-(C1-Pad1) -> Net-(J2-Pad2)
- J3 pad 3: Net-(J3-Pad3) -> /IOC_I2C_SCL
- J3 pad 4: /IOC_I2C_SCL -> Net-(C28-Pad1)
- J3 pad 5: Net-(J3-Pad5) -> /IOC_I2C_SCL
- J3 pad 6: /IOC_I2C_SDA -> Net-(C29-Pad2)
- J3 pad 7: /IOC_INT_INTA -> /IOC_I2C_SCL
- J3 pad 8: /IOC_~RESET -> /IOC_I2C_SCL
- K4 pad 1: Net-(K4-Pad1) -> Net-(C36-Pad1)
- K4 pad 2: Net-(C1-Pad2) -> Net-(J2-Pad2)
- K4 pad 5: Net-(C1-Pad2) -> Net-(J2-Pad2)
- K4 pad 8: Net-(K4-Pad8) -> Net-(C36-Pad2)
- L2 pad 1: +3V3 -> Net-(C16-Pad1)
- L2 pad 2: Net-(L2-Pad2) -> 1V65
- R10 pad 1: Net-(R10-Pad1) -> Net-(C54-Pad1)
- R11 pad 2: /Power Supply/1V65 -> Net-(C16-Pad1)
- R13 pad 2: Net-(R10-Pad1) -> Net-(R13-Pad2)
- R20 pad 1: Net-(D2-Pad2) -> Net-(R20-Pad1)
- R20 pad 2: Net-(R20-Pad2) -> Net-(D2-Pad2)
- R21 pad 1: Net-(D3-Pad2) -> Net-(R21-Pad1)
- R21 pad 2: Net-(R21-Pad2) -> Net-(D3-Pad2)
- R22 pad 1: Net-(D4-Pad2) -> Net-(R22-Pad1)
- R22 pad 2: Net-(R22-Pad2) -> Net-(D4-Pad2)
- R23 pad 1: Net-(D5-Pad2) -> Net-(R23-Pad1)
- R23 pad 2: Net-(R23-Pad2) -> Net-(D5-Pad2)
- R5 pad 1: Net-(C10-Pad1) -> Net-(C12-Pad1)
- R5 pad 2: Net-(R5-Pad2) -> Net-(C46-Pad2)
- R7 pad 1: Net-(C12-Pad1) -> Net-(C10-Pad1)
- R8 pad 1: /Power Supply/1V65 -> Net-(C16-Pad1)
- R8 pad 2: Net-(L2-Pad2) -> Net-(R8-Pad2)
- R9 pad 1: Net-(R5-Pad2) -> Net-(C46-Pad2)
- R9 pad 2: Net-(R12-Pad1) -> Net-(C46-Pad1)
- RF1 pad 1: Net-(C46-Pad1) -> /RFin
- T1 pad 1: Net-(C46-Pad2) -> /RFin
- T1 pad 4: /1V65 -> 1V65
- U11 pad 12: Net-(U11-Pad12) -> Net-(C50-Pad2)
- U11 pad 2: Net-(U11-Pad2) -> Net-(C51-Pad2)
- U11 pad 5: CLKI -> /Local oscillator/ALTLO_RX_CLKI
- U11 pad 6: Net-(U11-Pad12) -> Net-(R39-Pad1)
- U11 pad 8: CLKQ -> /Local oscillator/ALTLO_RX_CLKQ
- U11 pad 9: Net-(U11-Pad2) -> Net-(R40-Pad2)
- U2 pad 14: LO_CLK_I -> Net-(R34-Pad2)
- U2 pad 2: LO_CLK_Q -> Net-(R35-Pad2)
- U3 pad 1: Net-(R12-Pad1) -> Net-(C46-Pad1)
- U3 pad 2: Net-(R5-Pad2) -> Net-(C46-Pad2)
- U3 pad 7: Net-(R10-Pad1) -> Net-(C54-Pad1)
- U5 pad 14: /IOC_~RESET -> /IOC_I2C_SCL
- U5 pad 16: /IOC_INT_INTA -> /IOC_I2C_SCL
- U5 pad 9: /IOC_I2C_SDA -> /IOC_I2C_SCL
- U6 pad 12: /Local oscillator/LO_RX_QPH -> /Local oscillator/LO_RX_CLKQ
- U6 pad 13: /Local oscillator/LO_RX_IPH -> /Local oscillator/LO_RX_CLKI
- U6 pad 4: /Local oscillator/LO_I2C_SCL -> /IOC_I2C_SCL
- U6 pad 5: /Local oscillator/LO_I2C_SDA -> /IOC_I2C_SCL
- U6 pad 8: /Local oscillator/LO_TX_QPH -> /Local oscillator/LO_TX_CLKQ
- U6 pad 9: /Local oscillator/LO_TX_IPH -> /Local oscillator/LO_TX_CLKI
Routing:
- net GND: vias 3 -> 1
- net +3V3: vias 1 -> 0
- net (no net): vias 3 -> 1

Commit message: Update
Parts:
- moved TPQ1 66.9 mm to (-42.0, 14.0)
- moved TP6 65.5 mm to (6.00, 10.0)
- moved C53 61.5 mm to (-44.5, 9.00)
- moved C52 56.8 mm to (-44.5, 11.0), turned to 180 degrees
- moved TPI1 52.1 mm to (-42.0, 34.0), turned to 180 degrees
- moved R41 49.5 mm to (-37.0, 13.5), turned to 180 degrees
- moved TP5 47.0 mm to (-3.00, 10.0)
- moved R34 40.8 mm to (0.00, 9.00), turned to 270 degrees
- moved R44 27.3 mm to (-49.0, 22.0), turned to 180 degrees
- moved R45 24.0 mm to (-49.0, 19.0), turned to 180 degrees
- moved R42 21.1 mm to (-49.0, 16.0), turned to 180 degrees
- moved R43 21.0 mm to (-53.0, 17.0)
- moved C31 20.9 mm to (-44.5, -2.00), turned to 0 degrees
- moved C17 18.3 mm to (19.0, 29.5), turned to 90 degrees
- moved C30 18.1 mm to (-44.5, 0.00), turned to 180 degrees
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Connections:
- R8 pad 1: Net-(C16-Pad1) -> Net-(R8-Pad1)
- R8 pad 2: Net-(R8-Pad2) -> +3V3
- RV3 pad 1: +3V3 -> Net-(R8-Pad1)
- RV3 pad 2: +3V3 -> Net-(R8-Pad1)
- RV3 pad 3: Net-(R8-Pad2) -> Net-(C16-Pad1)
Routing:
- net (no net): vias 1 -> 2

Commit message: Update
Parts:
- removed TP18, TP19: TestPoint, TestPoint:TestPoint_Pad_D1.0mm
- added C55: 10n, Capacitor_SMD:C_0805_2012Metric, F.Cu at (11.0, 12.0)
- C14: value 4u7 -> 10u
- moved C1 54.1 mm to (11.0, 16.0), turned to 0 degrees
- moved TP13 42.9 mm to (-17.0, 13.0)
- moved TP15 41.0 mm to (-25.0, 14.5)
- moved R30 40.0 mm to (-22.0, 12.5), turned to 180 degrees
- moved TP12 28.6 mm to (-21.0, 15.0)
- moved C48 28.1 mm to (-18.0, 26.0), turned to 180 degrees
- moved C6 26.8 mm to (11.0, 14.0)
- moved C51 26.6 mm to (-5.00, -2.50)
- moved R39 19.4 mm to (-5.00, 3.00), turned to 180 degrees
- moved C50 19.3 mm to (-5.00, 5.50)
- moved TP11 19.3 mm to (0.50, 48.5)
- moved R37 17.4 mm to (4.50, 14.0), turned to 270 degrees
- moved R36 15.4 mm to (-1.50, 14.0), turned to 270 degrees
- moved TP14 15.3 mm to (-20.0, 32.5), turned to 180 degrees
- moved R40 15.3 mm to (-5.00, 0.00), turned to 180 degrees
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Connections:
- RV3 pad 1: Net-(R8-Pad1) -> Net-(C16-Pad1)
- RV3 pad 2: Net-(R8-Pad1) -> Net-(C16-Pad1)
- RV3 pad 3: Net-(C16-Pad1) -> Net-(R8-Pad1)
- T1 pad 1: /RFin -> GND
- T1 pad 2: GND -> /RFin
Routing:
- net /Filter/SIG_PRE_OUT: track 0.00 -> 50.8 mm
- net /Filter/SIG_PRE_IN: track 0.00 -> 42.1 mm
- net /Filter/SIG_LP_IN: track 0.00 -> 42.1 mm
- net /Filter/REL_COM: track 0.00 -> 42.0 mm
- net Net-(C2-Pad1): track 0.00 -> 17.5 mm
- net /RFin: track 0.00 -> 16.7 mm
- net Net-(C16-Pad1): track 0.00 -> 15.8 mm
- net Net-(C12-Pad1): track 9.92 -> 25.2 mm
- net Net-(C54-Pad1): track 0.00 -> 14.7 mm
- net Net-(C46-Pad1): track 0.00 -> 13.2 mm
- net +3V3: track 0.00 -> 12.4 mm, vias 0 -> 7
- net Net-(C40-Pad1): track 0.00 -> 12.2 mm
- net Net-(C8-Pad1): track 7.39 -> 19.5 mm
- net Net-(R2-Pad2): track 0.00 -> 10.6 mm
- net Net-(C10-Pad1): track 8.82 -> 19.3 mm
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- added copper zone on F.Cu, net +3V3

Commit message: Update
Parts:
- removed C50, C51: 10p, Capacitor_SMD:C_0805_2012Metric
- removed R39, R40: 1k, Resistor_SMD:R_0805_2012Metric
- removed R46, R47: 10, Resistor_SMD:R_0805_2012Metric
- added C56: 100n, Capacitor_SMD:C_0805_2012Metric, F.Cu at (-3.50, -2.00)
- J10, J11, J5, J6, J7, J8, J9: footprint Connector_PinSocket_1.27mm:PinSocket_1x04_P1.27mm_Vertical_SMD_Pin1Left -> Connector_PinSocket_1.27mm:PinSocket_1x04_P1.27mm_Vertical_SMD_Pin1Right
- J12, J13, J14, J15, J16, J17, J18, J19, J20, J21, J22, J23, J24, J25, J26, J27, J28, J29, J30, J31, J32: footprint Connector_PinSocket_1.27mm:PinSocket_1x03_P1.27mm_Vertical_SMD_Pin1Left -> Connector_PinSocket_1.27mm:PinSocket_1x03_P1.27mm_Vertical_SMD_Pin1Right
- moved D5 77.4 mm to (-27.8, 6.56)
- moved R23 77.2 mm to (-24.4, 8.56)
- moved R22 47.9 mm to (-27.8, 8.56)
- moved D4 43.7 mm to (-24.3, 6.56)
- moved R21 36.7 mm to (-20.9, 4.48)
- moved D3 36.4 mm to (-24.3, 4.52)
- moved D2 33.6 mm to (-27.8, 4.52)
- moved R20 32.0 mm to (-20.9, 6.43)
- moved R30 24.5 mm to (-17.0, 36.5)
- moved TP12 22.6 mm to (-14.0, 36.5)
- moved R31 22.5 mm to (-22.0, 14.5)
- moved R25 8.02 mm to (-11.5, 6.50), turned to 270 degrees
- moved R24 7.00 mm to (-9.00, 6.50)
- moved C38 6.50 mm to (-13.0, 2.00)
- moved R36 6.00 mm to (4.50, 14.0)
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Connections:
- J3 pad 3: /IOC_I2C_SCL -> /IOC_I2C_SDA
- J3 pad 7: /IOC_I2C_SCL -> /IOC_INT_INTA
- J3 pad 8: /IOC_I2C_SCL -> /IOC_~RESET
- R30 pad 2: Net-(R13-Pad2) -> Net-(R12-Pad1)
- R31 pad 2: Net-(R12-Pad1) -> Net-(R13-Pad2)
- U11 pad 12: Net-(C50-Pad2) -> Net-(U11-Pad12)
- U11 pad 2: Net-(C51-Pad2) -> Net-(U11-Pad2)
- U11 pad 5: /Local oscillator/ALTLO_RX_CLKI -> Net-(U11-Pad12)
- U11 pad 6: Net-(R39-Pad1) -> /Local oscillator/ALTLO_RX_CLKQ
- U11 pad 8: /Local oscillator/ALTLO_RX_CLKQ -> Net-(U11-Pad2)
- U11 pad 9: Net-(R40-Pad2) -> /Local oscillator/ALTLO_RX_CLKI
- U5 pad 14: /IOC_I2C_SCL -> /IOC_~RESET
- U5 pad 16: /IOC_I2C_SCL -> /IOC_INT_INTA
- U5 pad 9: /IOC_I2C_SCL -> /IOC_I2C_SDA
- U6 pad 5: /IOC_I2C_SCL -> /IOC_I2C_SDA
- U7 pad 14: /IOC_I2C_SCL -> /IOC_~RESET
- U7 pad 16: /IOC_I2C_SCL -> /IOC_INT_INTA
- U7 pad 9: /IOC_I2C_SCL -> /IOC_I2C_SDA
Routing:
- net GND: track 1.53 -> 151.0 mm, vias 3 -> 90
- net +3V3: track 12.4 -> 129.6 mm, vias 7 -> 35
- net /IOC_I2C_SDA: track 0.00 -> 62.8 mm, vias 0 -> 3
- net /IOC_I2C_SCL: track 0.00 -> 60.0 mm, vias 0 -> 3
- net /Filter/SIG_LP_OUT: track 0.00 -> 57.7 mm
- net Net-(C28-Pad1): track 5.66 -> 60.3 mm, vias 0 -> 5
- net /IOC_~RESET: track 0.00 -> 48.6 mm, vias 0 -> 3
- net Net-(C29-Pad2): track 5.66 -> 51.4 mm, vias 0 -> 5
- net Net-(J2-Pad2): track 0.00 -> 38.2 mm
- net /IOC_INT_INTA: track 0.00 -> 33.8 mm, vias 0 -> 4
- net /Filter/SIG_PRE_IN: track 42.1 -> 74.6 mm
- net /Local oscillator/LO_RX_CLKI: track 0.00 -> 14.5 mm
- net /Local oscillator/LO_RX_CLKQ: track 0.00 -> 13.8 mm
- net Net-(U10-Pad4): track 0.00 -> 12.5 mm, vias 0 -> 2
- net Net-(C36-Pad2): track 0.00 -> 11.7 mm, vias 0 -> 2
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- added copper zone on In2.Cu, net +3V3
- added copper zone on B.Cu, net GND
- added copper zone on F.Cu, net GND
- added copper zone on In1.Cu, net GND
Other:
- copper layers 2 -> 4
