File: Hardware/Bottom/GeckoTRX_Bottom.kicad_pcb (KiCad board)
At the start: 4 copper layers, 120 x 80 mm, 167 parts, among them J1 Jack-DC, J10 Conn_01x04_Female, J11 Conn_01x04_Female, J12 Conn_01x03_Female, J13 Conn_01x03_Female, J14 Conn_01x03_Female, J15 Conn_01x03_Female, J16 Conn_01x03_Female, J17 Conn_01x03_Female, J18 Conn_01x03_Female, J19 Conn_01x03_Female, J2 Conn_Coaxial, J20 Conn_01x03_Female, J21 Conn_01x03_Female, J22 Conn_01x03_Female, J23 Conn_01x03_Female, J24 Conn_01x03_Female, J25 Conn_01x03_Female, J26 Conn_01x03_Female, J27 Conn_01x03_Female, J28 Conn_01x03_Female, J29 Conn_01x03_Female, J3 Conn_02x05_Odd_Even, J30 Conn_01x03_Female, J31 Conn_01x03_Female, J32 Conn_01x03_Female, J4 Conn_02x05_Odd_Even, J5 Conn_01x04_Female, J6 Conn_01x04_Female, J7 Conn_01x04_Female, J8 Conn_01x04_Female, J9 Conn_01x04_Female, K4 G6K-2, T1 MABA-007237-ETC410, U1 TPS562200, U10 74LVC1G17, U11 74HC74D, U2 SN74CBTLV3253, U3 LT6231, U4 OP491-4, U5 MCP23017_ML, U6 Si5351A-B-GM, U7 MCP23017_ML, Y1 25MHz

Commit message: PCB v2 done
Parts:
- removed RV1: 100, Potentiometer_SMD:Potentiometer_Bourns_3224W_Vertical
- removed TPI1, TPQ1: TestPoint, TestPoint:TestPoint_Pad_D1.0mm
- added R39: 9k6, Resistor_SMD:R_0805_2012Metric, F.Cu at (-11.5, 16.0)
- added TP16: TestPoint, TestPoint:TestPoint_Pad_D1.0mm, F.Cu at (-42.0, 34.0)
- added TP17: TestPoint, TestPoint:TestPoint_Pad_D1.0mm, F.Cu at (-42.0, 14.0)
- C46, C54: value 15n -> 390p
- R10, R9: value 100 -> 10k
- R4, R5, R6, R7: value 100 -> 0R
- RV2: value 100 -> 2k
- RV3: value R_POT -> 2k
- TP10: value 180 -> TestPoint
- TP11: value GND -> TestPoint
- TP2: value RFin -> TestPoint
- TP3: value RFp -> TestPoint
- TP4: value RFn -> TestPoint
- TP5: value CLKI -> TestPoint
- TP6: value CLKQ -> TestPoint
- TP7: value 000 -> TestPoint
- TP8: value 090 -> TestPoint
- TP9: value 270 -> TestPoint
- moved R10 15.8 mm to (-14.5, 31.0), turned to 180 degrees
- moved C54 2.00 mm to (-9.50, 16.0)
Connections:
- R10 pad 1: Net-(C54-Pad1) -> Net-(C46-Pad2)
- R10 pad 2: Net-(C54-Pad2) -> Net-(C46-Pad1)
- RV2 pad 3: Net-(C54-Pad1) -> Net-(R39-Pad2)
Routing:
- net GND: track 167.5 -> 186.3 mm, vias 101 -> 287
- net Net-(R39-Pad2): track 0.00 -> 2.44 mm
- net Net-(C54-Pad1): track 19.0 -> 21.1 mm
- net Net-(C54-Pad2): track 11.2 -> 9.19 mm
- net /Filter/EN_PRE_TEST: track 80.2 -> 79.2 mm
Other:
- board text added: "Projektarbeit Version 0.2"

Commit message: keine ahnung, aber weitergemacht
Parts:
- added C1: 10n, Capacitor_SMD:C_0805_2012Metric, F.Cu at (10.5, 117.5)
- added C10: 15n, Capacitor_SMD:C_0805_2012Metric, F.Cu at (-4.00, 122.0)
- added C11: 1u, Capacitor_SMD:C_0805_2012Metric, F.Cu at (-18.0, 124.0)
- added C12: 15n, Capacitor_SMD:C_0805_2012Metric, F.Cu at (-4.00, 119.0)
- added C13: 1u, Capacitor_SMD:C_0805_2012Metric, F.Cu at (-44.0, 90.0)
- added C14: 10u, Capacitor_SMD:C_0805_2012Metric, F.Cu at (-46.0, 90.0)
- added C15: 100n, Capacitor_SMD:C_0805_2012Metric, F.Cu at (-48.0, 90.0)
- added C16: 10u, Capacitor_SMD:C_0805_2012Metric, F.Cu at (24.0, 132.0)
- added C17: 10u, Capacitor_SMD:C_0805_2012Metric, F.Cu at (28.0, 132.0)
- added C18: 68p, Capacitor_SMD:C_0805_2012Metric, F.Cu at (-22.0, 126.0)
- added C19: 68p, Capacitor_SMD:C_0805_2012Metric, F.Cu at (-22.0, 122.0)
- added C2: 10u, Capacitor_SMD:C_0805_2012Metric, F.Cu at (-46.0, 82.0)
- added C20: 100n, Capacitor_SMD:C_0805_2012Metric, F.Cu at (26.0, 132.0)
- added C21: 100n, Capacitor_SMD:C_0805_2012Metric, F.Cu at (15.0, 133.0)
- added C22: 680p, Capacitor_SMD:C_0805_2012Metric, F.Cu at (-26.0, 131.0)
- added C23: 680p, Capacitor_SMD:C_0805_2012Metric, F.Cu at (-26.0, 117.0)
- added C24: 10n, Capacitor_SMD:C_0805_2012Metric, F.Cu at (-18.0, 122.0)
- added C25: 10n, Capacitor_SMD:C_0805_2012Metric, F.Cu at (-22.0, 124.0)
- added C26: 22p, Capacitor_SMD:C_0805_2012Metric, F.Cu at (-35.0, 126.0)
- added C27: 22p, Capacitor_SMD:C_0805_2012Metric, F.Cu at (-35.0, 122.0)
- added C28: 470p, Capacitor_SMD:C_0805_2012Metric, F.Cu at (-35.0, 131.0)
- added C29: 470p, Capacitor_SMD:C_0805_2012Metric, F.Cu at (-35.0, 117.0)
- added C3: 10u, Capacitor_SMD:C_0805_2012Metric, F.Cu at (-44.0, 82.0)
- added C30: 1u, Capacitor_SMD:C_0805_2012Metric, F.Cu at (-44.5, 100.0)
- added C31: 100n, Capacitor_SMD:C_0805_2012Metric, F.Cu at (-44.5, 98.0)
- added C32: 1u, Capacitor_SMD:C_0805_2012Metric, F.Cu at (-7.00, 95.5)
- added C33: 100n, Capacitor_SMD:C_0805_2012Metric, F.Cu at (-14.5, 95.5)
- added C34: 100n, Capacitor_SMD:C_0805_2012Metric, F.Cu at (-12.0, 95.5)
- added C35: 100n, Capacitor_SMD:C_0805_2012Metric, F.Cu at (-9.50, 95.5)
- added C36: 100n, Capacitor_SMD:C_0805_2012Metric, F.Cu at (19.0, 73.0)
- added C37: 100n, Capacitor_SMD:C_0805_2012Metric, F.Cu at (-6.50, 106.5)
- added C38: 100n, Capacitor_SMD:C_0805_2012Metric, F.Cu at (-13.0, 102.0)
- added C4: 10u, Capacitor_SMD:C_0805_2012Metric, F.Cu at (-48.0, 82.0)
- added C44: 330u, Capacitor_SMD:C_Elec_6.3x7.7, F.Cu at (-38.0, 80.0)
- added C45: 330u, Capacitor_SMD:C_Elec_6.3x7.7, F.Cu at (-38.0, 88.0)
- added C46: 390p, Capacitor_SMD:C_0805_2012Metric, F.Cu at (-11.5, 132.0)
- added C5: 100n, Capacitor_SMD:C_0805_2012Metric, F.Cu at (-44.0, 86.0)
- added C56: 100n, Capacitor_SMD:C_0805_2012Metric, F.Cu at (-3.50, 98.0)
- added C6: 100n, Capacitor_SMD:C_0805_2012Metric, F.Cu at (10.5, 115.5)
- added C7: 100n, Capacitor_SMD:C_0805_2012Metric, F.Cu at (-51.0, 87.0)
- added C8: 15n, Capacitor_SMD:C_0805_2012Metric, F.Cu at (-4.00, 129.0)
- added C9: 15n, Capacitor_SMD:C_0805_2012Metric, F.Cu at (-4.00, 126.0)
- added D1: D, Diode_SMD:D_SMB, F.Cu at (-49.0, 76.0)
- added D2: LED, LED_SMD:LED_0805_2012Metric, F.Cu at (-86.2, -10.7)
- added D3: LED, LED_SMD:LED_0805_2012Metric, F.Cu at (-86.2, -8.69)
- added D4: LED, LED_SMD:LED_0805_2012Metric, F.Cu at (-82.7, -10.7)
- added D5: LED, LED_SMD:LED_0805_2012Metric, F.Cu at (-82.7, -8.69)
- added H1: MountingHole_Pad, MountingHole:MountingHole_3.2mm_M3_ISO14580_Pad, F.Cu at (-50.0, 70.0)
- added H2: MountingHole_Pad, MountingHole:MountingHole_3.2mm_M3_ISO14580_Pad, F.Cu at (50.0, 70.0)
- added H3: MountingHole_Pad, MountingHole:MountingHole_3.2mm_M3_ISO14580_Pad, F.Cu at (50.0, 130.0)
- added H4: MountingHole_Pad, MountingHole:MountingHole_3.2mm_M3_ISO14580_Pad, F.Cu at (-50.0, 130.0)
- added J1: Jack-DC, Connector_BarrelJack:BarrelJack_Wuerth_6941xx301002, F.Cu at (-40.0, 74.0)
- added J19: Conn_01x03_Female, Connector_PinSocket_1.27mm:PinSocket_1x03_P1.27mm_Vertical_SMD_Pin1Right, F.Cu at (27.0, 80.0)
- added J2: Conn_Coaxial, Connector_Coaxial:SMA_Molex_73251-1153_EdgeMount_Horizontal, F.Cu at (36.0, 65.0)
- added J20: Conn_01x03_Female, Connector_PinSocket_1.27mm:PinSocket_1x03_P1.27mm_Vertical_SMD_Pin1Right, F.Cu at (27.0, 87.0)
- added J21: Conn_01x03_Female, Connector_PinSocket_1.27mm:PinSocket_1x03_P1.27mm_Vertical_SMD_Pin1Right, F.Cu at (27.0, 94.0)
- added J22: Conn_01x03_Female, Connector_PinSocket_1.27mm:PinSocket_1x03_P1.27mm_Vertical_SMD_Pin1Right, F.Cu at (27.0, 101.0)
- added J23: Conn_01x03_Female, Connector_PinSocket_1.27mm:PinSocket_1x03_P1.27mm_Vertical_SMD_Pin1Right, F.Cu at (27.0, 108.0)
- added J24: Conn_01x03_Female, Connector_PinSocket_1.27mm:PinSocket_1x03_P1.27mm_Vertical_SMD_Pin1Right, F.Cu at (27.0, 115.0)
- added J25: Conn_01x03_Female, Connector_PinSocket_1.27mm:PinSocket_1x03_P1.27mm_Vertical_SMD_Pin1Right, F.Cu at (27.0, 122.0)
- added J26: Conn_01x03_Female, Connector_PinSocket_1.27mm:PinSocket_1x03_P1.27mm_Vertical_SMD_Pin1Right, F.Cu at (49.0, 80.0)
- added J27: Conn_01x03_Female, Connector_PinSocket_1.27mm:PinSocket_1x03_P1.27mm_Vertical_SMD_Pin1Right, F.Cu at (49.0, 87.0)
- added J28: Conn_01x03_Female, Connector_PinSocket_1.27mm:PinSocket_1x03_P1.27mm_Vertical_SMD_Pin1Right, F.Cu at (49.0, 94.0)
- added J29: Conn_01x03_Female, Connector_PinSocket_1.27mm:PinSocket_1x03_P1.27mm_Vertical_SMD_Pin1Right, F.Cu at (49.0, 101.0)
- added J3: Conn_02x05_Odd_Even, Connector_PinHeader_1.27mm:PinHeader_2x05_P1.27mm_Vertical_SMD, F.Cu at (-50.0, 97.0)
- added J30: Conn_01x03_Female, Connector_PinSocket_1.27mm:PinSocket_1x03_P1.27mm_Vertical_SMD_Pin1Right, F.Cu at (49.0, 108.0)
- added J31: Conn_01x03_Female, Connector_PinSocket_1.27mm:PinSocket_1x03_P1.27mm_Vertical_SMD_Pin1Right, F.Cu at (49.0, 115.0)
- added J32: Conn_01x03_Female, Connector_PinSocket_1.27mm:PinSocket_1x03_P1.27mm_Vertical_SMD_Pin1Right, F.Cu at (49.0, 122.0)
- added K1: G6K-2, Relay_SMD:Relay_DPDT_Omron_G6K-2G-Y, F.Cu at (-106.7, -6.47)
- added L1: 4u7, Inductor_SMD:L_Wuerth_MAPI-3015, F.Cu at (-47.0, 86.0)
- added L2: 33u, Inductor_SMD:L_0805_2012Metric, F.Cu at (15.0, 131.0)
- added R1: 10k, Resistor_SMD:R_0805_2012Metric, F.Cu at (-51.0, 81.1)
- added R10: 10k, Resistor_SMD:R_0805_2012Metric, F.Cu at (-14.5, 131.0)
- added R11: 2k, Resistor_SMD:R_0805_2012Metric, F.Cu at (30.0, 132.0)
- added R12: 6k8, Resistor_SMD:R_0805_2012Metric, F.Cu at (-22.0, 131.0)
- added R13: 6k8, Resistor_SMD:R_0805_2012Metric, F.Cu at (-22.0, 117.0)
- added R14: 150k, Resistor_SMD:R_0805_2012Metric, F.Cu at (-22.0, 128.5)
- added R15: 150k, Resistor_SMD:R_0805_2012Metric, F.Cu at (-22.0, 119.5)
- added R2: 10k, Resistor_SMD:R_0805_2012Metric, F.Cu at (-52.0, 90.0)
- added R20: 100, Resistor_SMD:R_0805_2012Metric, F.Cu at (-79.3, -8.82)
- added R21: 100, Resistor_SMD:R_0805_2012Metric, F.Cu at (-86.2, -6.69)
- added R22: 100, Resistor_SMD:R_0805_2012Metric, F.Cu at (-79.3, -10.8)
- added R23: 100, Resistor_SMD:R_0805_2012Metric, F.Cu at (-82.8, -6.69)
- added R24: 10k, Resistor_SMD:R_0805_2012Metric, F.Cu at (-9.00, 106.5)
- added R25: DNP, Resistor_SMD:R_0805_2012Metric, F.Cu at (-11.5, 106.5)
- added R26: DNP, Resistor_SMD:R_0805_2012Metric, F.Cu at (-14.0, 106.5)
- added R3: 54k9, Resistor_SMD:R_0805_2012Metric, F.Cu at (-50.0, 90.0)
- added R4: 0R, Resistor_SMD:R_0805_2012Metric, F.Cu at (-8.50, 126.0)
- added R42: 50, Resistor_SMD:R_1206_3216Metric, F.Cu at (-49.0, 116.0)
- added R43: 0R, Resistor_SMD:R_0402_1005Metric, F.Cu at (-53.0, 117.0)
- added R44: 50, Resistor_SMD:R_1206_3216Metric, F.Cu at (-49.0, 122.0)
- added R45: 50, Resistor_SMD:R_1206_3216Metric, F.Cu at (-49.0, 119.0)
- added R5: 0R, Resistor_SMD:R_0805_2012Metric, F.Cu at (-8.50, 129.0)
- added R6: 0R, Resistor_SMD:R_0805_2012Metric, F.Cu at (-8.50, 122.0)
- added R7: 0R, Resistor_SMD:R_0805_2012Metric, F.Cu at (-8.50, 119.0)
- added R8: 1k, Resistor_SMD:R_0805_2012Metric, F.Cu at (25.0, 129.0)
- added R9: 10k, Resistor_SMD:R_0805_2012Metric, F.Cu at (-9.50, 132.0)
- added RV1: 2k, Potentiometer_SMD:Potentiometer_Bourns_3224W_Vertical, F.Cu at (-85.3, -0.12)
- added RV2: 2k, Potentiometer_SMD:Potentiometer_Bourns_3224W_Vertical, F.Cu at (-15.5, 117.0)
- added T1: MABA-007237-ETC410, Transformer_SMD:Transformer_MACOM_SM-22, F.Cu at (10.0, 131.0)
- added TP11: TestPoint, TestPoint:TestPoint_Pad_D1.0mm, F.Cu at (-6.00, 132.0)
- added TP2: TestPoint, TestPoint:TestPoint_Pad_D1.0mm, F.Cu at (18.0, 125.0)
- added TP3: TestPoint, TestPoint:TestPoint_Pad_D1.0mm, F.Cu at (2.00, 130.5)
- added TP4: TestPoint, TestPoint:TestPoint_Pad_D1.0mm, F.Cu at (5.50, 130.5)
- added TP5: TestPoint, TestPoint:TestPoint_Pad_D1.0mm, F.Cu at (4.50, 117.0)
- added TP6: TestPoint, TestPoint:TestPoint_Pad_D1.0mm, F.Cu at (1.50, 117.0)
- added TP7: TestPoint, TestPoint:TestPoint_Pad_D1.0mm, F.Cu at (10.5, 119.5)
- added TP8: TestPoint, TestPoint:TestPoint_Pad_D1.0mm, F.Cu at (10.5, 122.0)
- added U1: TPS562200, Package_TO_SOT_SMD:SOT-23-6, F.Cu at (-51.0, 84.0)
- added U2: SN74CBTLV3253, Package_SO:SOIC-16_3.9x9.9mm_P1.27mm, F.Cu at (3.00, 124.0)
- added U3: LT6231, Package_SO:SOIC-8_3.9x4.9mm_P1.27mm, F.Cu at (-13.5, 124.0)
- added U4: OP491-4, Package_SO:SOIC-14_3.9x8.7mm_P1.27mm, F.Cu at (-28.5, 124.0)
- added U5: MCP23017_ML, Package_DFN_QFN:QFN-28-1EP_6x6mm_P0.65mm_EP4.25x4.25mm, F.Cu at (-38.0, 97.0)
- added U6: Si5351A-B-GM, Package_DFN_QFN:QFN-20-1EP_4x4mm_P0.5mm_EP2.7x2.7mm, F.Cu at (-7.50, 101.0)
- added Y1: 25MHz, Crystal:Crystal_SMD_Abracon_ABM10-4Pin_2.5x2.0mm, F.Cu at (-13.0, 99.0)
- moved C39 100.0 mm to (7.00, 96.5)
- moved C40 100.0 mm to (12.0, 103.5)
- moved C41 100.0 mm to (9.50, 96.5)
- moved C42 100.0 mm to (-0.50, 95.5)
- moved C43 100.0 mm to (3.50, 95.5)
- moved C47 100.0 mm to (15.0, 129.0)
- moved C48 100.0 mm to (-18.0, 126.0)
- moved C52 100.0 mm to (-44.5, 111.0)
- moved C53 100.0 mm to (-44.5, 109.0)
- moved C54 100.0 mm to (-9.50, 116.0)
- moved C55 100.0 mm to (10.5, 113.5)
- moved IOUT1 100.0 mm to (-42.0, 129.0)
- moved J10 100.0 mm to (5.00, 87.0)
- moved J11 100.0 mm to (12.0, 87.0)
- moved J12 100.0 mm to (-30.0, 66.0)
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Connections:
- C39 pad 1: +3V3 -> (no net)
- C39 pad 2: GND -> (no net)
- C40 pad 1: Net-(C40-Pad1) -> (no net)
- C40 pad 2: Net-(C40-Pad2) -> (no net)
- C41 pad 1: GND -> (no net)
- C41 pad 2: +3V3 -> (no net)
- C42 pad 1: +3V3 -> (no net)
- C42 pad 2: GND -> (no net)
- C43 pad 1: GND -> (no net)
- C43 pad 2: +3V3 -> (no net)
- C47 pad 1: 1V65 -> (no net)
- C47 pad 2: GND -> (no net)
- C48 pad 1: +3V3 -> (no net)
- C48 pad 2: GND -> (no net)
- C52 pad 1: +3V3 -> (no net)
- C52 pad 2: GND -> (no net)
- C53 pad 1: GND -> (no net)
- C53 pad 2: +3V3 -> (no net)
- C54 pad 1: Net-(C54-Pad1) -> (no net)
- C54 pad 2: Net-(C54-Pad2) -> (no net)
- C55 pad 1: +3V3 -> (no net)
- C55 pad 2: GND -> (no net)
- IOUT1 pad 1: Net-(C28-Pad1) -> (no net)
- IOUT1 pad 2: GND -> (no net)
- J10 pad 1: /Filter/SIG_LP_IN -> (no net)
- J10 pad 2: GND -> (no net)
- J10 pad 3: /Filter/REL_COM -> (no net)
- J10 pad 4: /Filter/SW_LP_10 -> (no net)
- J11 pad 1: /Filter/SIG_LP_IN -> (no net)
- J11 pad 2: GND -> (no net)
- J11 pad 3: /Filter/REL_COM -> (no net)
- J11 pad 4: /Filter/SW_LP_CUST -> (no net)
- J12 pad 1: /Filter/SIG_LP_OUT -> (no net)
- J12 pad 2: GND -> (no net)
- J12 pad 3: GND -> (no net)
- J13 pad 1: /Filter/SIG_LP_OUT -> (no net)
- J13 pad 2: GND -> (no net)
- J13 pad 3: GND -> (no net)
- J14 pad 1: /Filter/SIG_LP_OUT -> (no net)
- J14 pad 2: GND -> (no net)
- J14 pad 3: GND -> (no net)
- J15 pad 1: /Filter/SIG_LP_OUT -> (no net)
- J15 pad 2: GND -> (no net)
- J15 pad 3: GND -> (no net)
- J16 pad 1: /Filter/SIG_LP_OUT -> (no net)
- J16 pad 2: GND -> (no net)
- J16 pad 3: GND -> (no net)
- J17 pad 1: /Filter/SIG_LP_OUT -> (no net)
- J17 pad 2: GND -> (no net)
- J17 pad 3: GND -> (no net)
- J18 pad 1: /Filter/SIG_LP_OUT -> (no net)
- J18 pad 2: GND -> (no net)
- J18 pad 3: GND -> (no net)
- J4 pad 1: Net-(J4-Pad1) -> (no net)
- J4 pad 10: /I2C_LO_SDA -> (no net)
- J4 pad 2: /ADC_SPI_CLK -> (no net)
- J4 pad 3: Net-(J4-Pad3) -> (no net)
- J4 pad 4: /ADC_SPI_MISO -> (no net)
- J4 pad 5: Net-(J4-Pad5) -> (no net)
- J4 pad 6: /ADC_SPI_CS -> (no net)
- J4 pad 7: Net-(J4-Pad7) -> (no net)
- J4 pad 8: /I2C_LO_SCL -> (no net)
- J4 pad 9: Net-(J4-Pad9) -> (no net)
- J5 pad 1: /Filter/SIG_LP_IN -> (no net)
- J5 pad 2: GND -> (no net)
- J5 pad 3: /Filter/REL_COM -> (no net)
- J5 pad 4: /Filter/SW_LP_160 -> (no net)
- J6 pad 1: /Filter/SIG_LP_IN -> (no net)
- J6 pad 2: GND -> (no net)
- J6 pad 3: /Filter/REL_COM -> (no net)
- J6 pad 4: /Filter/SW_LP_80 -> (no net)
- J7 pad 1: /Filter/SIG_LP_IN -> (no net)
- J7 pad 2: GND -> (no net)
- J7 pad 3: /Filter/REL_COM -> (no net)
- J7 pad 4: /Filter/SW_LP_40 -> (no net)
- J8 pad 1: /Filter/SIG_LP_IN -> (no net)
- J8 pad 2: GND -> (no net)
- J8 pad 3: /Filter/REL_COM -> (no net)
- J8 pad 4: /Filter/SW_LP_20 -> (no net)
- J9 pad 1: /Filter/SIG_LP_IN -> (no net)
- J9 pad 2: GND -> (no net)
- J9 pad 3: /Filter/REL_COM -> (no net)
- J9 pad 4: /Filter/SW_LP_15 -> (no net)
- K4 pad 1: Net-(C36-Pad1) -> (no net)
- K4 pad 2: Net-(J2-Pad2) -> (no net)
- K4 pad 3: /Filter/SIG_PRE_IN -> (no net)
- K4 pad 4: GND -> (no net)
- K4 pad 5: Net-(J2-Pad2) -> (no net)
- K4 pad 6: /Filter/SIG_LP_OUT -> (no net)
- K4 pad 7: GND -> (no net)
- K4 pad 8: Net-(C36-Pad2) -> (no net)
- LO1 pad 1: Net-(C40-Pad2) -> (no net)
- LO1 pad 2: GND -> (no net)
- QOUT1 pad 1: Net-(C29-Pad2) -> (no net)
- QOUT1 pad 2: GND -> (no net)
- R16 pad 1: Net-(C22-Pad2) -> (no net)
- R16 pad 2: Net-(C28-Pad2) -> (no net)
- R17 pad 1: Net-(C29-Pad1) -> (no net)
- R17 pad 2: Net-(C23-Pad1) -> (no net)
- R18 pad 1: Net-(C28-Pad2) -> (no net)
- R18 pad 2: Net-(C26-Pad1) -> (no net)
- R19 pad 1: Net-(C29-Pad1) -> (no net)
- R19 pad 2: Net-(C27-Pad1) -> (no net)
- R27 pad 1: Net-(C40-Pad1) -> (no net)
- R27 pad 2: +3V3 -> (no net)
- R28 pad 1: GND -> (no net)
- R28 pad 2: Net-(C40-Pad1) -> (no net)
- R29 pad 1: GND -> (no net)
- R29 pad 2: Net-(C40-Pad1) -> (no net)
- R30 pad 1: Net-(C46-Pad1) -> (no net)
- R30 pad 2: Net-(R12-Pad1) -> (no net)
- R31 pad 1: Net-(C54-Pad1) -> (no net)
- R31 pad 2: Net-(R13-Pad2) -> (no net)
- R32 pad 1: /GPIO Expander/GPIO_1 -> (no net)
- R32 pad 2: Net-(C36-Pad1) -> (no net)
- R33 pad 1: /GPIO Expander/GPIO_0 -> (no net)
- R33 pad 2: Net-(C36-Pad2) -> (no net)
- R34 pad 1: /Local oscillator/ALTLO_RX_CLKI -> (no net)
- R34 pad 2: Net-(R34-Pad2) -> (no net)
- R35 pad 1: /Local oscillator/ALTLO_RX_CLKQ -> (no net)
- R35 pad 2: Net-(R35-Pad2) -> (no net)
- R36 pad 1: /Local oscillator/LO_RX_CLKI -> (no net)
- R36 pad 2: Net-(R34-Pad2) -> (no net)
- R37 pad 1: /Local oscillator/LO_RX_CLKQ -> (no net)
- R37 pad 2: Net-(R35-Pad2) -> (no net)
- R38 pad 1: /Filter/SIG_PRE_OUT -> (no net)
- R38 pad 2: /RFin -> (no net)
- R39 pad 1: Net-(C54-Pad1) -> (no net)
- R39 pad 2: Net-(R39-Pad2) -> (no net)
- R41 pad 1: +3V3 -> (no net)
- R41 pad 2: Net-(R41-Pad2) -> (no net)
- RF1 pad 1: /RFin -> (no net)
- RF1 pad 2: GND -> (no net)
- RV3 pad 1: Net-(C16-Pad1) -> (no net)
- RV3 pad 2: Net-(C16-Pad1) -> (no net)
- RV3 pad 3: Net-(R8-Pad1) -> (no net)
- TP1 pad 1: Net-(C40-Pad1) -> (no net)
- TP10 pad 1: Net-(C12-Pad1) -> (no net)
- TP12 pad 1: Net-(C46-Pad1) -> (no net)
- TP13 pad 1: Net-(C54-Pad1) -> (no net)
- TP14 pad 1: Net-(R12-Pad1) -> (no net)
- TP15 pad 1: Net-(R13-Pad2) -> (no net)
- TP16 pad 1: Net-(C28-Pad1) -> (no net)
- TP17 pad 1: Net-(C29-Pad2) -> (no net)
- TP9 pad 1: Net-(C10-Pad1) -> (no net)
- U10 pad 2: Net-(C40-Pad1) -> (no net)
- U10 pad 3: GND -> (no net)
- U10 pad 4: Net-(U10-Pad4) -> (no net)
- U10 pad 5: +3V3 -> (no net)
- U11 pad 1: +3V3 -> (no net)
- U11 pad 10: +3V3 -> (no net)
- U11 pad 11: Net-(U10-Pad4) -> (no net)
- U11 pad 12: Net-(U11-Pad12) -> (no net)
- U11 pad 13: +3V3 -> (no net)
- U11 pad 14: +3V3 -> (no net)
- U11 pad 2: Net-(U11-Pad2) -> (no net)
- U11 pad 3: Net-(U10-Pad4) -> (no net)
- U11 pad 4: +3V3 -> (no net)
- U11 pad 5: Net-(U11-Pad12) -> (no net)
- U11 pad 6: /Local oscillator/ALTLO_RX_CLKQ -> (no net)
- U11 pad 7: GND -> (no net)
- U11 pad 8: Net-(U11-Pad2) -> (no net)
- U11 pad 9: /Local oscillator/ALTLO_RX_CLKI -> (no net)
- U7 pad 1: /GPIO Expander/GPIO_4 -> (no net)
- U7 pad 10: Net-(U7-Pad10) -> (no net)
- U7 pad 11: Net-(R41-Pad2) -> (no net)
- U7 pad 12: GND -> (no net)
- U7 pad 13: GND -> (no net)
- U7 pad 14: /IOC_~RESET -> (no net)
- U7 pad 15: Net-(U7-Pad15) -> (no net)
- U7 pad 16: /IOC_INT_INTA -> (no net)
- U7 pad 17: /GPIO Expander/GPIO_8 -> (no net)
- U7 pad 18: /GPIO Expander/GPIO_9 -> (no net)
- U7 pad 19: /GPIO Expander/GPIO_10 -> (no net)
- U7 pad 2: /GPIO Expander/GPIO_5 -> (no net)
- U7 pad 20: /GPIO Expander/GPIO_11 -> (no net)
- U7 pad 21: /GPIO Expander/GPIO_12 -> (no net)
- U7 pad 22: /GPIO Expander/GPIO_13 -> (no net)
- U7 pad 23: /GPIO Expander/GPIO_14 -> (no net)
- U7 pad 24: /GPIO Expander/GPIO_15 -> (no net)
- U7 pad 25: /GPIO Expander/GPIO_0 -> (no net)
- U7 pad 26: /GPIO Expander/GPIO_1 -> (no net)
- U7 pad 27: /GPIO Expander/GPIO_2 -> (no net)
- U7 pad 28: /GPIO Expander/GPIO_3 -> (no net)
- U7 pad 29: GND -> (no net)
- U7 pad 3: /GPIO Expander/GPIO_6 -> (no net)
- U7 pad 4: /GPIO Expander/GPIO_7 -> (no net)
- U7 pad 5: +3V3 -> (no net)
- U7 pad 6: GND -> (no net)
- U7 pad 7: Net-(U7-Pad7) -> (no net)
- U7 pad 8: /IOC_I2C_SCL -> (no net)
- U7 pad 9: /IOC_I2C_SDA -> (no net)
Routing:
- net (no net): track 0.00 -> 2657.2 mm, vias 0 -> 409
- net +3V3: track 138.6 -> 113.8 mm, vias 39 -> 35
- net Net-(C40-Pad1): track 21.1 -> 0.00 mm
- net Net-(U10-Pad4): track 12.5 -> 0.00 mm, vias 2 -> 0
- net Net-(C40-Pad2): track 12.4 -> 0.00 mm, vias 2 -> 0
- net /Local oscillator/ALTLO_RX_CLKI: track 10.9 -> 0.00 mm
- net /Local oscillator/ALTLO_RX_CLKQ: track 10.8 -> 0.00 mm
- net Net-(U11-Pad2): track 10.4 -> 0.00 mm, vias 2 -> 0
- net GND: track 186.3 -> 178.8 mm, vias 287 -> 277
- net Net-(U11-Pad12): track 6.45 -> 0.00 mm
- added copper zone on B.Cu, net (none)
- added copper zone on F.Cu, net (none)
- added copper zone on In1.Cu, net (none)
- added copper zone on In2.Cu, net (none)
Other:
- board size 120 x 80 mm -> 120 x 180 mm
